File: pcb/usb/mini/mini.kicad_sch (KiCad schematic)
At the start: 2 parts, among them J1 USB_B_Mini, U1 CH340C

Commit message: Signed-off-by: Dmitry Ponyatov <dponyatov@samsa.local>
Connections:
- net VCC5: now reaches J1.1 (VBUS)
Changed lines of the file:
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@@
   (junction (at 82.55 101.6) (diameter 0) (color 0 0 0 0)
+  )
+  (junction (at 92.71 83.82) (diameter 0) (color 0 0 0 0)
   )
   (wire (pts (xy 80.01 99.06) (xy 80.01 101.6))
@@
   )
   (wire (pts (xy 125.73 87.63) (xy 129.54 87.63))
+    (stroke (width 0) (type default) (color 0 0 0 0))
+  )
+  (wire (pts (xy 90.17 83.82) (xy 92.71 83.82))
+    (stroke (width 0) (type default) (color 0 0 0 0))
+  )
+  (wire (pts (xy 92.71 73.66) (xy 92.71 83.82))
     (stroke (width 0) (type default) (color 0 0 0 0))
   )
@@
   )
   (wire (pts (xy 139.7 102.87) (xy 139.7 106.68))
+    (stroke (width 0) (type default) (color 0 0 0 0))
+  )
+  (wire (pts (xy 92.71 83.82) (xy 96.52 83.82))
     (stroke (width 0) (type default) (color 0 0 0 0))
   )
@@
     (effects (font (size 1.27 1.27)) (justify right bottom))
   )
+  (global_label "VCC5" (shape input) (at 92.71 73.66 90) (fields_autoplaced)
+    (effects (font (size 1.27 1.27)) (justify left))
+    (property "Intersheet References" "${INTERSHEET_REFS}" (id 0) (at 92.6306 66.4088 90)
+      (effects (font (size 1.27 1.27)) (justify left) hide)
+    )
+  )
   (symbol (lib_id "power:GND") (at 139.7 106.68 0) (unit 1)

Commit message: Signed-off-by: Dmitry Ponyatov <dponyatov@samsa.local>
Parts:
- added J?: Conn_01x06_Male, symbol Connector:Conn_01x06_Male
- J?: renamed from J1; symbol Connector:USB_B_Mini -> connector:USB_B_Mini
Changed lines of the file:
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@@
     )
+  )
+  (symbol (lib_id "Connector:Conn_01x06_Male") (at 175.26 82.55 0) (mirror y) (unit 1)
+    (in_bom yes) (on_board yes) (fields_autoplaced)
+    (property "Reference" "J?" (id 0) (at 176.53 82.5499 0)
+      (effects (font (size 1.27 1.27)) (justify right))
+    )
+    (property "Value" "Conn_01x06_Male" (id 1) (at 176.53 85.0899 0)
+      (effects (font (size 1.27 1.27)) (justify right))
+    )
+    (property "Footprint" "" (id 2) (at 175.26 82.55 0)
+      (effects (font (size 1.27 1.27)) hide)
+    )
+    (property "Datasheet" "~" (id 3) (at 175.26 82.55 0)
+      (effects (font (size 1.27 1.27)) hide)
+    )
+    (pin "1")
+    (pin "2")
+    (pin "3")
+    (pin "4")
+    (pin "5")
+    (pin "6")
   )
   (symbol (lib_id "power:GND") (at 139.7 106.68 0) (unit 1)
@@
     (pin "1")
   )
-  (symbol (lib_id "Connector:USB_B_Mini") (at 82.55 88.9 0) (unit 1)
+  (symbol (lib_id "connector:USB_B_Mini") (at 82.55 88.9 0) (unit 1)
     (in_bom yes) (on_board yes) (fields_autoplaced)
-    (property "Reference" "J1" (id 0) (at 82.55 76.2 0))
-    (property "Value" "USB_B_Mini" (id 1) (at 82.55 78.74 0))
+    (property "Reference" "J?" (id 0) (at 77.47 77.47 0)
+      (effects (font (size 1.27 1.27)) (justify left))
+    )
+    (property "Value" "USB_B_Mini" (id 1) (at 77.47 80.01 0)
+      (effects (font (size 1.27 1.27)) (justify left))
+    )
     (property "Footprint" "connector:USB_Mini-B_DS1104" (id 2) (at 86.36 90.17 0)
       (effects (font (size 1.27 1.27)) hide)
@@
       (reference "#PWR0102") (unit 1) (value "GND") (footprint "")
     )
+    (path "/aa0eaef1-e2de-4828-9cb9-7fe98fa29c67"
+      (reference "J?") (unit 1) (value "Conn_01x06_Male") (footprint "")
+    )
     (path "/ce1752a3-7b9b-4e5d-a7cf-dfe02fc97064"
-      (reference "J1") (unit 1) (value "USB_B_Mini") (footprint "connector:USB_Mini-B_DS1104")
+      (reference "J?") (unit 1) (value "USB_B_Mini") (footprint "connector:USB_Mini-B_DS1104")
     )
     (path "/e3c48a62-3601-400c-9094-a10797422302"

Commit message: Signed-off-by: Dmitry Ponyatov <dponyatov@samsa.local>
Parts:
- added J2: Conn_01x03, symbol Connector_Generic:Conn_01x03
- added U2: AMS1117-3.3, Package_TO_SOT_SMD:SOT-223-3_TabPin2, symbol Regulator_Linear:AMS1117-3.3
- J3: renamed from J?; value Conn_01x06_Male -> Conn_01x10_Male; symbol Connector:Conn_01x06_Male -> Connector:Conn_01x10_Male
- gave numbers to parts that had none: 1
Connections:
- net GND: now also J3.10 (Pin_10), U2.1 (GND)
- net VCC5: now also J2.1 (Pin_1), U2.3 (VI)
- net TxD: now reaches J3.1 (Pin_1)
- net TxD: now also U1.2 (TXD)
- net RxD: now reaches J3.2 (Pin_2)
- net RxD: now also U1.3 (RXD)
- net CTS: now reaches J3.4 (Pin_4)
- net CTS: now also U1.9 (~{CTS})
- net DSR: now reaches J3.5 (Pin_5)
- net DSR: now also U1.10 (~{DSR})
- net RI: now reaches J3.6 (Pin_6)
- net RI: now also U1.11 (~{RI})
- net DCD: now reaches U1.12 (~{DCD})
- net DCD: now also J3.7 (Pin_7)
- net DTR: now reaches U1.13 (~{DTR})
- net DTR: now also J3.8 (Pin_8)
- net RTS: now reaches U1.14 (~{RTS})
- net RTS: now also J3.9 (Pin_9)
- net at U1.16 (VCC): now also J2.2 (Pin_2), J2.3 (Pin_3), U2.2 (VO)

Commit message: Signed-off-by: Dmitry Ponyatov <dponyatov@samsa.local>
Parts:
- J?: renamed from J1; value USB_B_Mini -> M-1J; symbol connector:USB_B_Mini -> connector:M-1J
Changed lines of the file:
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@@
     (pin "1")
   )
-  (symbol (lib_id "connector:USB_B_Mini") (at 82.55 88.9 0) (unit 1)
+  (symbol (lib_id "connector:M-1J") (at 82.55 88.9 0) (unit 1)
     (in_bom yes) (on_board yes) (fields_autoplaced)
-    (property "Reference" "J1" (id 0) (at 77.47 77.47 0)
+    (property "Reference" "J?" (id 0) (at 77.47 77.47 0)
       (effects (font (size 1.27 1.27)) (justify left))
     )
-    (property "Value" "USB_B_Mini" (id 1) (at 77.47 80.01 0)
+    (property "Value" "M-1J" (id 1) (at 77.47 80.01 0)
       (effects (font (size 1.27 1.27)) (justify left))
     )
@@
       (reference "#PWR0103") (unit 1) (value "GND") (footprint "")
     )
-    (path "/ce1752a3-7b9b-4e5d-a7cf-dfe02fc97064"
-      (reference "J1") (unit 1) (value "USB_B_Mini") (footprint "connector:USB_Mini-B_DS1104")
-    )
     (path "/7e516f75-6c1a-4b57-b7bc-2c21da4bc555"
       (reference "J2") (unit 1) (value "Conn_01x03") (footprint "")
@@
       (reference "J3") (unit 1) (value "Conn_01x10_Male") (footprint "")
     )
+    (path "/ce1752a3-7b9b-4e5d-a7cf-dfe02fc97064"
+      (reference "J?") (unit 1) (value "M-1J") (footprint "connector:USB_Mini-B_DS1104")
+    )
     (path "/e3c48a62-3601-400c-9094-a10797422302"

Commit message: Signed-off-by: Dmitry Ponyatov <dponyatov@samsa.local>
Parts:
- added U?: MAX485ED, smd:SOP-8_3.76x4.96mm_P1.27mm, symbol ic:MAX485ED
- gave numbers to parts that had none: 1
Connections:
- net GND: now also U?.5 (GND)
- net RxD: now also U?.1 (RO)
- net TxD: now also U?.4 (DI)
- net at J2.2 (Pin_2), U1.16 (VCC): now also U?.8 (VCC); no longer J2.3 (Pin_3), U2.2 (VO)
- new net: J2.3 (Pin_3), U2.2 (VO)
Changed lines of the file:
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@@
   (junction (at 97.79 69.85) (diameter 0) (color 0 0 0 0)
   )
-  (junction (at 124.46 50.8) (diameter 0) (color 0 0 0 0)
-  )
   (junction (at 139.7 66.04) (diameter 0) (color 0 0 0 0)
   )
@@
     (stroke (width 0) (type default) (color 0 0 0 0))
   )
+  (wire (pts (xy 212.09 66.04) (xy 212.09 72.39))
+    (stroke (width 0) (type default) (color 0 0 0 0))
+  )
   (wire (pts (xy 125.73 87.63) (xy 129.54 87.63))
     (stroke (width 0) (type default) (color 0 0 0 0))
@@
     (stroke (width 0) (type default) (color 0 0 0 0))
   )
+  (wire (pts (xy 194.31 82.55) (xy 201.93 82.55))
+    (stroke (width 0) (type default) (color 0 0 0 0))
+  )
+  (wire (pts (xy 194.31 90.17) (xy 201.93 90.17))
+    (stroke (width 0) (type default) (color 0 0 0 0))
+  )
   (wire (pts (xy 149.86 77.47) (xy 170.18 77.47))
     (stroke (width 0) (type default) (color 0 0 0 0))
   )
+  (wire (pts (xy 194.31 85.09) (xy 201.93 85.09))
+    (stroke (width 0) (type default) (color 0 0 0 0))
+  )
   (wire (pts (xy 90.17 83.82) (xy 92.71 83.82))
     (stroke (width 0) (type default) (color 0 0 0 0))
   )
+  (wire (pts (xy 212.09 100.33) (xy 212.09 104.14))
+    (stroke (width 0) (type default) (color 0 0 0 0))
+  )
   (wire (pts (xy 97.79 69.85) (xy 97.79 76.2))
     (stroke (width 0) (type default) (color 0 0 0 0))
@@
     (stroke (width 0) (type default) (color 0 0 0 0))
   )
-  (wire (pts (xy 124.46 50.8) (xy 139.7 50.8))
-    (stroke (width 0) (type default) (color 0 0 0 0))
-  )
   (wire (pts (xy 149.86 95.25) (xy 170.18 95.25))
     (stroke (width 0) (type default) (color 0 0 0 0))
   )
+  (wire (pts (xy 139.7 66.04) (xy 212.09 66.04))
+    (stroke (width 0) (type default) (color 0 0 0 0))
+  )
   (wire (pts (xy 109.22 69.85) (xy 97.79 69.85))
     (stroke (width 0) (type default) (color 0 0 0 0))
@@
     (stroke (width 0) (type default) (color 0 0 0 0))
   )
-  (wire (pts (xy 139.7 50.8) (xy 139.7 66.04))
-    (stroke (width 0) (type default) (color 0 0 0 0))
-  )
   (wire (pts (xy 92.71 83.82) (xy 96.52 83.82))
     (stroke (width 0) (type default) (color 0 0 0 0))
   )
   (wire (pts (xy 97.79 76.2) (xy 92.71 76.2))
+    (stroke (width 0) (type default) (color 0 0 0 0))
+  )
+  (wire (pts (xy 194.31 87.63) (xy 201.93 87.63))
     (stroke (width 0) (type default) (color 0 0 0 0))
   )
@@
     (effects (font (size 1.27 1.27)) (justify left bottom))
   )
+  (label "TxD" (at 195.58 90.17 0)
+    (effects (font (size 1.27 1.27)) (justify left bottom))
+  )
   (label "DCD" (at 165.1 92.71 0)
+    (effects (font (size 1.27 1.27)) (justify left bottom))
+  )
+  (label "RxD" (at 195.58 82.55 0)
     (effects (font (size 1.27 1.27)) (justify left bottom))
   )
@@
       (effects (font (size 1.27 1.27)) (justify left) hide)
     )
+  )
+  (symbol (lib_id "ic:MAX485ED") (at 212.09 85.09 0) (unit 1)
+    (in_bom yes) (on_board yes) (fields_autoplaced)
+    (property "Reference" "U?" (id 0) (at 205.994 73.66 0))
+    (property "Value" "MAX485ED" (id 1) (at 212.852 73.66 0)
+      (effects (font (size 1.27 1.27)) (justify left))
+    )
+    (property "Footprint" "smd:SOP-8_3.76x4.96mm_P1.27mm" (id 2) (at 212.09 102.87 0)
+      (effects (font (size 1.27 1.27)) hide)
+    )
+    (property "Datasheet" "https://datasheets.maximintegrated.com/en/ds/MAX1487E-MAX491E.pdf" (id 3) (at 212.09 83.82 0)
+      (effects (font (size 1.27 1.27)) hide)
+    )
+    (pin "1")
+    (pin "2")
+    (pin "3")
+    (pin "4")
+    (pin "5")
+    (pin "6")
+    (pin "7")
+    (pin "8")
+  )
+  (symbol (lib_id "power:GND") (at 212.09 104.14 0) (unit 1)
+    (in_bom yes) (on_board yes) (fields_autoplaced)
+    (property "Reference" "#PWR?" (id 0) (at 212.09 110.49 0)
+      (effects (font (size 1.27 1.27)) hide)
+    )
+    (property "Value" "GND" (id 1) (at 212.09 109.22 0))
+    (property "Footprint" "" (id 2) (at 212.09 104.14 0)
+      (effects (font (size 1.27 1.27)) hide)
+    )
+    (property "Datasheet" "" (id 3) (at 212.09 104.14 0)
+      (effects (font (size 1.27 1.27)) hide)
+    )
+    (pin "1")
   )
   (symbol (lib_id "Regulator_Linear:AMS1117-3.3") (at 111.76 50.8 0) (unit 1)
@@
   (symbol (lib_id "connector:M-1J") (at 82.55 88.9 0) (unit 1)
     (in_bom yes) (on_board yes) (fields_autoplaced)
-    (property "Reference" "J?" (id 0) (at 77.47 77.47 0)
+    (property "Reference" "J1" (id 0) (at 77.47 77.47 0)
       (effects (font (size 1.27 1.27)) (justify left))
     )
@@
       (reference "#PWR0103") (unit 1) (value "GND") (footprint "")
     )
+    (path "/469bbc30-0f91-4fdc-8782-c8d961e33467"
+      (reference "#PWR?") (unit 1) (value "GND") (footprint "")
+    )
+    (path "/ce1752a3-7b9b-4e5d-a7cf-dfe02fc97064"
+      (reference "J1") (unit 1) (value "M-1J") (footprint "connector:USB_Mini-B_DS1104")
+    )
     (path "/7e516f75-6c1a-4b57-b7bc-2c21da4bc555"
       (reference "J2") (unit 1) (value "Conn_01x03") (footprint "")
@@
       (reference "J3") (unit 1) (value "Conn_01x10_Male") (footprint "")
     )
-    (path "/ce1752a3-7b9b-4e5d-a7cf-dfe02fc97064"
-      (reference "J?") (unit 1) (value "M-1J") (footprint "connector:USB_Mini-B_DS1104")
-    )
     (path "/e3c48a62-3601-400c-9094-a10797422302"
       (reference "U1") (unit 1) (value "CH340C") (footprint "Package_SO:SOIC-16_3.9x9.9mm_P1.27mm")
@@
       (reference "U2") (unit 1) (value "AMS1117-3.3") (footprint "Package_TO_SOT_SMD:SOT-223-3_TabPin2")
     )
-  )
+    (path "/0cfa8113-056e-4664-b8b8-022625e2ed47"
+      (reference "U?") (unit 1) (value "MAX485ED") (footprint "smd:SOP-8_3.76x4.96mm_P1.27mm")
+    )
+  )

Commit message: Signed-off-by: Dmitry Ponyatov <dponyatov@samsa.local>
Parts:
- removed U?: MAX485ED, smd:SOP-8_3.76x4.96mm_P1.27mm, symbol ic:MAX485ED
- added C1, C2: 10uF, smd:C_0805, symbol Device:C_Small
- added J4: Conn_01x04_Male, Connector_PinHeader_2.54mm:PinHeader_1x04_P2.54mm_Horizontal, symbol Connector:Conn_01x04_Male
- J2: footprint (none) -> connector:PinHeader_1x03_P2.54mm_Vertical
- J3: value Conn_01x10_Male -> Conn_01x08; footprint (none) -> Connector_PinHeader_2.54mm:PinHeader_1x08_P2.54mm_Horizontal; symbol Connector:Conn_01x10_Male -> Connector_Generic:Conn_01x08
Connections:
- net CTS: now also J3.2 (Pin_2); no longer J3.4 (Pin_4)
- net DCD: now also J3.5 (Pin_5); no longer J3.7 (Pin_7)
- net DSR: now also J3.3 (Pin_3); no longer J3.5 (Pin_5)
- net DTR: now also J3.6 (Pin_6); no longer J3.8 (Pin_8)
- net GND: now also J3.1 (Pin_1), C1.2, C2.2, J4.1 (Pin_1); no longer J3.10 (Pin_10)
- net RI: now also J3.4 (Pin_4); no longer J3.6 (Pin_6)
- net RTS: now also J3.7 (Pin_7); no longer J3.9 (Pin_9)
- net RxD: now also J4.3 (Pin_3); no longer J3.2 (Pin_2)
- net TxD: now also J4.2 (Pin_2); no longer J3.1 (Pin_1)
- net VCC5: now also C1.1
- net VCCIO: now reaches J2.2 (Pin_2), U1.16 (VCC)
- net VCCIO: now also J4.4 (Pin_4)
- net VCC3: now reaches J2.3 (Pin_3), U2.2 (VO)
- net VCC3: now also J3.8 (Pin_8), C2.1
- no-connect marks 0 -> 1
Other:
- moved on the sheet: U1
