File: pcb/usb/mini/mini.kicad_sch (KiCad schematic)
At the start: 2 parts, among them J1 USB_B_Mini, U1 CH340C

Commit message: Signed-off-by: Dmitry Ponyatov <dponyatov@gmail.com>
Changed lines of the file:
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@@
   )
   (symbol (lib_id "Interface_USB:CH340C") (at 139.7 87.63 0) (unit 1)
-    (in_bom yes) (on_board yes) (fields_autoplaced)
-    (property "Reference" "U1" (id 0) (at 141.7194 102.87 0)
+    (in_bom yes) (on_board yes)
+    (property "Reference" "U1" (id 0) (at 142.24 72.39 0)
       (effects (font (size 1.27 1.27)) (justify left))
     )
-    (property "Value" "CH340C" (id 1) (at 141.7194 105.41 0)
+    (property "Value" "CH340C" (id 1) (at 140.97 102.87 0)
       (effects (font (size 1.27 1.27)) (justify left))
     )

Commit message: Signed-off-by: Dmitry Ponyatov <dponyatov@gmail.com>
Parts:
- added C1, C2: 10uF, smd:C_0805, symbol Device:C_Small
- added J2: Conn_01x03, connector:PinHeader_1x03_P2.54mm_Vertical, symbol Connector_Generic:Conn_01x03
- added J3: Conn_01x08, Connector_PinHeader_2.54mm:PinHeader_1x08_P2.54mm_Horizontal, symbol Connector_Generic:Conn_01x08
- added J4: Conn_01x04_Male, Connector_PinHeader_2.54mm:PinHeader_1x04_P2.54mm_Horizontal, symbol Connector:Conn_01x04_Male
- added U2: AMS1117-3.3, Package_TO_SOT_SMD:SOT-223-3_TabPin2, symbol Regulator_Linear:AMS1117-3.3
- J1: value USB_B_Mini -> M-1J; symbol Connector:USB_B_Mini -> connector:M-1J
Connections:
- net GND: now also C1.2, C2.2, J3.1 (Pin_1), J4.1 (Pin_1), U2.1 (GND)
- net VCC5: now also C1.1, J2.1 (Pin_1), U2.3 (VI)
- net DSR: now reaches U1.10 (~{DSR})
- net DSR: now also J3.3 (Pin_3)
- net RI: now reaches U1.11 (~{RI})
- net RI: now also J3.4 (Pin_4)
- net DCD: now reaches U1.12 (~{DCD})
- net DCD: now also J3.5 (Pin_5)
- net DTR: now reaches U1.13 (~{DTR})
- net DTR: now also J3.6 (Pin_6)
- net RTS: now reaches U1.14 (~{RTS})
- net RTS: now also J3.7 (Pin_7)
- net VCCIO: now reaches U1.16 (VCC)
- net VCCIO: now also J2.2 (Pin_2), J4.4 (Pin_4)
- net TxD: now reaches U1.2 (TXD)
- net TxD: now also J4.2 (Pin_2)
- net RxD: now reaches U1.3 (RXD)
- net RxD: now also J4.3 (Pin_3)
- net CTS: now reaches U1.9 (~{CTS})
- net CTS: now also J3.2 (Pin_2)
- new net VCC3: C2.1, J2.3 (Pin_3), J3.8 (Pin_8), U2.2 (VO)
- no-connect marks 0 -> 1
Other:
- moved on the sheet: U1
