File: pcb/usb/mini/mini.kicad_pcb (KiCad board)
At the start: 2 copper layers, 50.8 x 25.4 mm, 2 parts, among them J1 USB_B_Mini, U1 CH340C

Commit message: Signed-off-by: Dmitry Ponyatov <dponyatov@samsa.local>
Connections:
- J1 pad 1: unconnected-(J1-Pad1) -> VCC5
Changed lines of the file:
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@@
   )
   (net 0 "")
-  (net 1 "unconnected-(J1-Pad1)")
+  (net 1 "VCC5")
   (net 2 "/D-")
   (net 3 "/D+")
@@
     (pad "" np_thru_hole circle (at -2.2 0 270) (size 0.9 0.9) (drill 0.9) (layers *.Cu *.Mask))
     (pad "1" smd rect (at -1.6 -2.6 270) (size 0.5 2.5) (layers "F.Cu" "F.Paste" "F.Mask")
-      (net 1 "unconnected-(J1-Pad1)") (pinfunction "VBUS") (pintype "power_out"))
+      (net 1 "VCC5") (pinfunction "VBUS") (pintype "power_out"))
     (pad "2" smd rect (at -0.8 -2.6 270) (size 0.5 2.5) (layers "F.Cu" "F.Paste" "F.Mask")
       (net 2 "/D-") (pinfunction "D-") (pintype "bidirectional"))

Commit message: Signed-off-by: Dmitry Ponyatov <dponyatov@samsa.local>
Routing:
- net GND: track 35.5 -> 40.0 mm
Other:
- outline, holes or cut-outs redrawn

Commit message: Signed-off-by: Dmitry Ponyatov <dponyatov@samsa.local>
Parts:
- added U2: AMS1117-3.3, Package_TO_SOT_SMD:SOT-223-3_TabPin2, F.Cu at (144.3, 85.1)
- moved U1 2.06 mm to (154.4, 90.5)
Connections:
- U1 pad 10: unconnected-(U1-Pad10) -> /DSR
- U1 pad 11: unconnected-(U1-Pad11) -> /RI
- U1 pad 12: unconnected-(U1-Pad12) -> /DCD
- U1 pad 13: unconnected-(U1-Pad13) -> /DTR
- U1 pad 14: unconnected-(U1-Pad14) -> /RTS
- U1 pad 16: unconnected-(U1-Pad16) -> Net-(U1-Pad16)
- U1 pad 2: unconnected-(U1-Pad2) -> /TxD
- U1 pad 3: unconnected-(U1-Pad3) -> /RxD
- U1 pad 9: unconnected-(U1-Pad9) -> /CTS
Routing:
- net Net-(U1-Pad16): track 0.00 -> 10.7 mm
- net GND: track 40.0 -> 48.2 mm
- net VCC5: track 0.00 -> 5.18 mm
- net /D+: track 19.0 -> 21.1 mm
- net /D-: track 20.6 -> 22.7 mm

Commit message: Signed-off-by: Dmitry Ponyatov <dponyatov@samsa.local>
Parts:
- J1: value USB_B_Mini -> M-1J
- moved U2 0.76 mm to (144.3, 85.9)
Routing:
- net Net-(U1-Pad16): track 10.7 -> 10.2 mm

Commit message: Signed-off-by: Dmitry Ponyatov <dponyatov@samsa.local>
Parts:
- added U3: MAX485ED, smd:SOP-8_3.76x4.96mm_P1.27mm, F.Cu at (167.6, 88.9)
Connections:
- U1 pad 16: Net-(U1-Pad16) -> Net-(J2-Pad2)
- U2 pad 2: Net-(U1-Pad16) -> Net-(J2-Pad3)
Routing:
- net Net-(U1-Pad16): track 10.2 -> 0.00 mm
- net Net-(J2-Pad3): track 0.00 -> 10.2 mm
Changed lines of the file:
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@@
   (net 15 "/RTS")
   (net 16 "unconnected-(U1-Pad15)")
-  (net 17 "Net-(U1-Pad16)")
+  (net 17 "Net-(J2-Pad2)")
   (net 18 "GND")
+  (net 19 "Net-(J2-Pad3)")
+  (net 20 "unconnected-(U3-Pad2)")
+  (net 21 "unconnected-(U3-Pad3)")
+  (net 22 "unconnected-(U3-Pad6)")
+  (net 23 "unconnected-(U3-Pad7)")
   (footprint "Package_SO:SOIC-16_3.9x9.9mm_P1.27mm" (layer "F.Cu")
     (at 154.4326 90.5203 90)
@@
       (net 16 "unconnected-(U1-Pad15)") (pinfunction "R232") (pintype "input"))
     (pad "16" smd roundrect (at 2.475 -4.445 90) (size 1.95 0.6) (layers "F.Cu" "F.Paste" "F.Mask") (roundrect_rratio 0.25)
-      (net 17 "Net-(U1-Pad16)") (pinfunction "VCC") (pintype "power_in"))
+      (net 17 "Net-(J2-Pad2)") (pinfunction "VCC") (pintype "power_in"))
     (model "${KICAD6_3DMODEL_DIR}/Package_SO.3dshapes/SOIC-16_3.9x9.9mm_P1.27mm.wrl"
       (offset (xyz 0 0 0))
@@
       (net 18 "GND") (pinfunction "GND") (pintype "power_in"))
     (pad "2" smd rect (at 3.15 0) (size 2 3.8) (layers "F.Cu" "F.Paste" "F.Mask")
-      (net 17 "Net-(U1-Pad16)") (pinfunction "VO") (pintype "power_out"))
+      (net 19 "Net-(J2-Pad3)") (pinfunction "VO") (pintype "power_out"))
     (pad "2" smd rect (at -3.15 0) (size 2 1.5) (layers "F.Cu" "F.Paste" "F.Mask")
-      (net 17 "Net-(U1-Pad16)") (pinfunction "VO") (pintype "power_out"))
+      (net 19 "Net-(J2-Pad3)") (pinfunction "VO") (pintype "power_out"))
     (pad "3" smd rect (at -3.15 2.3) (size 2 1.5) (layers "F.Cu" "F.Paste" "F.Mask")
       (net 1 "VCC5") (pinfunction "VI") (pintype "power_in"))
@@
     )
   )
+  (footprint "smd:SOP-8_3.76x4.96mm_P1.27mm" (layer "F.Cu")
+    (at 167.64 88.9)
+    (descr "SOP, 8 Pin (https://ww2.minicircuits.com/case_style/XX211.pdf), generated with kicad-footprint-generator ipc_gullwing_generator.py")
+    (tags "SOP SO")
+    (property "Sheetfile" "mini.kicad_sch")
+    (property "Sheetname" "")
+    (attr smd)
+    (fp_text reference "U3" (at 0 -3.43) (layer "F.SilkS")
+      (effects (font (size 1 1) (thickness 0.15)))
+    )
+    (fp_text value "MAX485ED" (at 0 3.43) (layer "F.Fab")
+      (effects (font (size 1 1) (thickness 0.15)))
+    )
+    (fp_text user "${REFERENCE}" (at 0 0) (layer "F.Fab")
+      (effects (font (size 0.94 0.94) (thickness 0.14)))
+    )
+    (fp_line (start 0 -2.59) (end -3.525 -2.59) (layer "F.SilkS") (width 0.12))
+    (fp_line (start 0 2.59) (end -1.88 2.59) (layer "F.SilkS") (width 0.12))
+    (fp_line (start 0 2.59) (end 1.88 2.59) (layer "F.SilkS") (width 0.12))
+    (fp_line (start 0 -2.59) (end 1.88 -2.59) (layer "F.SilkS") (width 0.12))
+    (fp_line (start -3.78 2.73) (end 3.78 2.73) (layer "F.CrtYd") (width 0.05))
+    (fp_line (start -3.78 -2.73) (end -3.78 2.73) (layer "F.CrtYd") (width 0.05))
+    (fp_line (start 3.78 2.73) (end 3.78 -2.73) (layer "F.CrtYd") (width 0.05))
+    (fp_line (start 3.78 -2.73) (end -3.78 -2.73) (layer "F.CrtYd") (width 0.05))
+    (fp_line (start -1.88 -1.54) (end -0.94 -2.48) (layer "F.Fab") (width 0.1))
+    (fp_line (start 1.88 2.48) (end -1.88 2.48) (layer "F.Fab") (width 0.1))
+    (fp_line (start 1.88 -2.48) (end 1.88 2.48) (layer "F.Fab") (width 0.1))
+    (fp_line (start -0.94 -2.48) (end 1.88 -2.48) (layer "F.Fab") (width 0.1))
+    (fp_line (start -1.88 2.48) (end -1.88 -1.54) (layer "F.Fab") (width 0.1))
+    (pad "1" smd roundrect (at -2.5375 -1.905) (size 1.975 0.65) (layers "F.Cu" "F.Paste" "F.Mask") (roundrect_rratio 0.25)
+      (net 6 "/RxD") (pinfunction "RO") (pintype "output"))
+    (pad "2" smd roundrect (at -2.5375 -0.635) (size 1.975 0.65) (layers "F.Cu" "F.Paste" "F.Mask") (roundrect_rratio 0.25)
+      (net 20 "unconnected-(U3-Pad2)") (pinfunction "~{RE}") (pintype "input"))
+    (pad "3" smd roundrect (at -2.5375 0.635) (size 1.975 0.65) (layers "F.Cu" "F.Paste" "F.Mask") (roundrect_rratio 0.25)
+      (net 21 "unconnected-(U3-Pad3)") (pinfunction "DE") (pintype "input"))
+    (pad "4" smd roundrect (at -2.5375 1.905) (size 1.975 0.65) (layers "F.Cu" "F.Paste" "F.Mask") (roundrect_rratio 0.25)
+      (net 5 "/TxD") (pinfunction "DI") (pintype "input"))
+    (pad "5" smd roundrect (at 2.5375 1.905) (size 1.975 0.65) (layers "F.Cu" "F.Paste" "F.Mask") (roundrect_rratio 0.25)
+      (net 18 "GND") (pinfunction "GND") (pintype "power_in"))
+    (pad "6" smd roundrect (at 2.5375 0.635) (size 1.975 0.65) (layers "F.Cu" "F.Paste" "F.Mask") (roundrect_rratio 0.25)
+      (net 22 "unconnected-(U3-Pad6)") (pinfunction "A") (pintype "bidirectional"))
+    (pad "7" smd roundrect (at 2.5375 -0.635) (size 1.975 0.65) (layers "F.Cu" "F.Paste" "F.Mask") (roundrect_rratio 0.25)
+      (net 23 "unconnected-(U3-Pad7)") (pinfunction "B") (pintype "bidirectional"))
+    (pad "8" smd roundrect (at 2.5375 -1.905) (size 1.975 0.65) (layers "F.Cu" "F.Paste" "F.Mask") (roundrect_rratio 0.25)
+      (net 17 "Net-(J2-Pad2)") (pinfunction "VCC") (pintype "power_in"))
+    (model "${KICAD6_3DMODEL_DIR}/Package_SO.3dshapes/SOP-8_3.76x4.96mm_P1.27mm.wrl"
+      (offset (xyz 0 0 0))
+      (scale (xyz 1 1 1))
+      (rotate (xyz 0 0 0))
+    )
+  )
   (gr_line (start 127 101.346) (end 127 76.454) (layer "Edge.Cuts") (width 0.1))
   (gr_line (start 177.546 101.6) (end 127.254 101.6) (layer "Edge.Cuts") (width 0.1))
@@
   (segment (start 135.95 88.9) (end 137.2 88.9) (width 0.5) (layer "F.Cu") (net 3))
   (segment (start 154.7948 92.0882) (end 155.0676 92.9953) (width 0.5) (layer "F.Cu") (net 3))
-  (segment (start 148.5318 87.1915) (end 148.422 87.0817) (width 0.5) (layer "F.Cu") (net 17))
-  (segment (start 141.872 85.852) (end 142.122 85.852) (width 0.5) (layer "F.Cu") (net 17))
-  (segment (start 149.6927 87.1915) (end 148.5318 87.1915) (width 0.5) (layer "F.Cu") (net 17))
-  (segment (start 148.172 87.0817) (end 147.422 85.852) (width 0.5) (layer "F.Cu") (net 17))
-  (segment (start 141.122 85.852) (end 141.872 85.852) (width 0.5) (layer "F.Cu") (net 17))
-  (segment (start 149.9876 88.0453) (end 149.6927 87.1915) (width 0.5) (layer "F.Cu") (net 17))
-  (segment (start 142.122 85.852) (end 146.422 85.852) (width 0.5) (layer "F.Cu") (net 17))
-  (segment (start 148.422 87.0817) (end 148.172 87.0817) (width 0.5) (layer "F.Cu") (net 17))
-  (segment (start 146.672 85.852) (end 147.422 85.852) (width 0.5) (layer "F.Cu") (net 17))
-  (segment (start 146.422 85.852) (end 146.672 85.852) (width 0.5) (layer "F.Cu") (net 17))
   (segment (start 136.95 92.3) (end 136.95 92.0235) (width 0.5) (layer "F.Cu") (net 18))
   (segment (start 134.4141 85.25) (end 134.3254 85.3387) (width 0.5) (layer "F.Cu") (net 18))
@@
   (segment (start 140.372 84.026) (end 141.122 83.552) (width 0.5) (layer "F.Cu") (net 18))
   (segment (start 149.937 92.4203) (end 149.687 92.4203) (width 0.5) (layer "F.Cu") (net 18))
+  (segment (start 148.5318 87.1915) (end 148.422 87.0817) (width 0.5) (layer "F.Cu") (net 19))
+  (segment (start 141.872 85.852) (end 142.122 85.852) (width 0.5) (layer "F.Cu") (net 19))
+  (segment (start 149.6927 87.1915) (end 148.5318 87.1915) (width 0.5) (layer "F.Cu") (net 19))
+  (segment (start 148.172 87.0817) (end 147.422 85.852) (width 0.5) (layer "F.Cu") (net 19))
+  (segment (start 141.122 85.852) (end 141.872 85.852) (width 0.5) (layer "F.Cu") (net 19))
+  (segment (start 149.9876 88.0453) (end 149.6927 87.1915) (width 0.5) (layer "F.Cu") (net 19))
+  (segment (start 142.122 85.852) (end 146.422 85.852) (width 0.5) (layer "F.Cu") (net 19))
+  (segment (start 148.422 87.0817) (end 148.172 87.0817) (width 0.5) (layer "F.Cu") (net 19))
+  (segment (start 146.672 85.852) (end 147.422 85.852) (width 0.5) (layer "F.Cu") (net 19))
+  (segment (start 146.422 85.852) (end 146.672 85.852) (width 0.5) (layer "F.Cu") (net 19))
 )

Commit message: Signed-off-by: Dmitry Ponyatov <dponyatov@samsa.local>
Parts:
- removed U3: MAX485ED, smd:SOP-8_3.76x4.96mm_P1.27mm
- added C1: 10uF, smd:C_0805, F.Cu at (140.3, 85.5)
- added C2: 10uF, smd:C_0805, F.Cu at (141.0, 82.2)
- added J2: Conn_01x03, connector:PinHeader_1x03_P2.54mm_Vertical, F.Cu at (144.8, 88.9)
- added J3: Conn_01x08, Connector_PinHeader_2.54mm:PinHeader_1x08_P2.54mm_Horizontal, B.Cu at (171.7, 83.1)
- added J4: Conn_01x04_Male, Connector_PinHeader_2.54mm:PinHeader_1x04_P2.54mm_Horizontal, B.Cu at (170.6, 96.8)
- moved U1 4.48 mm to (155.1, 95.0)
- moved U2 3.60 mm to (146.7, 83.2)
Connections:
- U1 pad 16: Net-(J2-Pad2) -> /VCCIO
- U2 pad 2: Net-(J2-Pad3) -> /VCC3
Routing:
- net /TxD: track 0.00 -> 23.5 mm
- net /RxD: track 0.00 -> 22.0 mm
- net /VCC3: track 0.00 -> 18.0 mm
- net /VCCIO: track 0.00 -> 15.7 mm, vias 0 -> 2
- net /CTS: track 0.00 -> 14.6 mm
- net /DSR: track 0.00 -> 14.2 mm
- net GND: track 47.9 -> 34.3 mm, vias 0 -> 1
- net /RI: track 0.00 -> 13.2 mm
- net /DCD: track 0.00 -> 12.1 mm
- net /DTR: track 0.00 -> 11.9 mm
- net /RTS: track 0.00 -> 11.2 mm
- net Net-(J2-Pad3): track 10.2 -> 0.00 mm
- net VCC5: track 5.47 -> 14.1 mm
- net /D-: track 22.7 -> 25.8 mm
- net /D+: track 21.1 -> 23.9 mm
- added copper zone on B.Cu, net GND

Commit message: Signed-off-by: Dmitry Ponyatov <dponyatov@samsa.local>
Routing:
- net /VCCIO: track 15.7 -> 32.3 mm
Changed lines of the file:
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@@
     (aux_axis_origin 127 101.6)
     (pcbplotparams
-      (layerselection 0x00010fc_ffffffff)
+      (layerselection 0x0000000_fffffffe)
       (disableapertmacros false)
       (usegerberextensions false)
@@
       (svguseinch false)
       (svgprecision 6)
-      (excludeedgelayer true)
+      (excludeedgelayer false)
       (plotframeref false)
       (viasonmask false)
@@
     (fp_line (start 1.27 6.35) (end -1.27 6.35) (layer "F.Fab") (width 0.1))
     (fp_line (start -1.27 6.35) (end -1.27 -0.635) (layer "F.Fab") (width 0.1))
-    (pad "1" thru_hole roundrect (at 0 0 90) (size 2 2) (drill 0.8) (layers *.Cu *.Mask) (roundrect_rratio 0.25)
+    (pad "1" thru_hole rect (at 0 0 90) (size 2 2) (drill 0.8) (layers *.Cu *.Mask)
       (net 1 "VCC5") (pinfunction "Pin_1") (pintype "passive"))
     (pad "2" thru_hole circle (at 0 2.54 90) (size 2 2) (drill 0.8) (layers *.Cu *.Mask)
@@
     (fp_line (start 10.04 0.32) (end 10.04 -0.32) (layer "B.Fab") (width 0.1))
     (fp_line (start 10.04 -4.76) (end 10.04 -5.4) (layer "B.Fab") (width 0.1))
-    (pad "1" thru_hole roundrect (at 0 0) (size 2 2) (drill 1) (layers *.Cu *.Mask) (roundrect_rratio 0.25)
+    (pad "1" thru_hole rect (at 0 0) (size 2 2) (drill 1) (layers *.Cu *.Mask)
       (net 17 "GND") (pinfunction "Pin_1") (pintype "passive"))
     (pad "2" thru_hole oval (at 0 -2.54) (size 1.7 1.7) (drill 1) (layers *.Cu *.Mask)
@@
   (gr_line (start 127 101.346) (end 127.254 101.6) (layer "Edge.Cuts") (width 0.1))
   (gr_line (start 177.546 76.2) (end 177.8 76.454) (layer "Edge.Cuts") (width 0.1))
-  (segment (start 144.399 88.9) (end 143.51 88.011) (width 0.5) (layer "F.Cu") (net 1))
-  (segment (start 143.51 88.011) (end 143.51 85.51) (width 0.5) (layer "F.Cu") (net 1))
+  (segment (start 143.51 85.51) (end 143.535 85.485) (width 0.5) (layer "F.Cu") (net 1))
   (segment (start 143.535 85.485) (end 144.014 85.985) (width 0.5) (layer "F.Cu") (net 1))
   (segment (start 143.5101 85.5099) (end 143.535 85.485) (width 0.5) (layer "F.Cu") (net 1))
@@
   (segment (start 141.285 85.5099) (end 141.536 85.4974) (width 0.5) (layer "F.Cu") (net 1))
   (segment (start 141.285 86.553) (end 141.285 85.5099) (width 0.5) (layer "F.Cu") (net 1))
-  (segment (start 144.795 88.9) (end 144.399 88.9) (width 0.5) (layer "F.Cu") (net 1))
-  (segment (start 143.51 85.51) (end 143.535 85.485) (width 0.5) (layer "F.Cu") (net 1))
+  (segment (start 144.795 88.9) (end 143.51 87.615) (width 0.5) (layer "F.Cu") (net 1))
+  (segment (start 143.51 87.615) (end 143.51 85.51) (width 0.5) (layer "F.Cu") (net 1))
   (segment (start 140.538 87.3) (end 141.285 86.553) (width 0.5) (layer "F.Cu") (net 1))
   (segment (start 141.285 85.5099) (end 143.5101 85.5099) (width 0.5) (layer "F.Cu") (net 1))
@@
   (via (at 163.068 92.456) (size 1.2) (drill 0.5) (layers "F.Cu" "B.Cu") (free) (net 19))
   (via (at 147.32 92.456) (size 1.2) (drill 0.5) (layers "F.Cu" "B.Cu") (free) (net 19))
+  (segment (start 162.052 91.44) (end 163.068 92.456) (width 0.5) (layer "B.Cu") (net 19))
+  (segment (start 148.336 91.44) (end 162.052 91.44) (width 0.5) (layer "B.Cu") (net 19))
+  (segment (start 147.32 92.456) (end 148.336 91.44) (width 0.5) (layer "B.Cu") (net 19))
   (zone (net 17) (net_name "GND") (layer "B.Cu") (name "GND") (hatch none 0.508)
     (connect_pads (clearance 0.5))
