File: pcb/usb/mini/mini.kicad_pcb (KiCad board)
At the start: 2 copper layers, 50.8 x 25.4 mm, 2 parts, among them J1 USB_B_Mini, U1 CH340C

Commit message: Signed-off-by: Dmitry Ponyatov <dponyatov@gmail.com>
Parts:
- moved J1 1.27 mm to (134.6, 88.9)
Other:
- outline, holes or cut-outs redrawn
Changed lines of the file:
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@@
       (effects (font (size 1 1) (thickness 0.15)))
     )
-    (fp_text user "${REFERENCE}" (at 0 0 90) (layer "F.Fab")
+    (fp_text user "${REFERENCE}" (at 0 2.54 90) (layer "F.Fab")
       (effects (font (size 0.98 0.98) (thickness 0.15)))
     )
@@
     )
   )
-  (footprint "connector:USB_Mini-B_DS1104" (layer "F.Cu")
-    (at 133.35 88.9 -90)
+  (footprint "connector:USB_Mini-B_DS1104" locked (layer "F.Cu")
+    (at 134.62 88.9 -90)
     (descr "Mini USB 2.0 Type B SMT Horizontal 5 Contacts")
     (tags "Mini USB 2.0 Type B")
@@
     (fp_line (start -1.6 -2.85) (end -1.3 -3.35) (layer "F.Fab") (width 0.1))
     (fp_line (start -1.3 -3.35) (end 3.85 -3.35) (layer "F.Fab") (width 0.1))
-    (pad "" np_thru_hole circle (at 2.2 0 270) (size 0.9 0.9) (drill 0.9) (layers *.Cu *.Mask))
-    (pad "" np_thru_hole circle (at -2.2 0 270) (size 0.9 0.9) (drill 0.9) (layers *.Cu *.Mask))
-    (pad "1" smd rect (at -1.6 -2.6 270) (size 0.5 2.5) (layers "F.Cu" "F.Paste" "F.Mask")
+    (pad "" np_thru_hole circle locked (at 2.2 0 270) (size 0.9 0.9) (drill 0.9) (layers *.Cu *.Mask))
+    (pad "" np_thru_hole circle locked (at -2.2 0 270) (size 0.9 0.9) (drill 0.9) (layers *.Cu *.Mask))
+    (pad "1" smd rect locked (at -1.6 -2.6 270) (size 0.5 2.5) (layers "F.Cu" "F.Paste" "F.Mask")
       (net 1 "VCC5") (pinfunction "VBUS") (pintype "power_out"))
-    (pad "2" smd rect (at -0.8 -2.6 270) (size 0.5 2.5) (layers "F.Cu" "F.Paste" "F.Mask")
+    (pad "2" smd rect locked (at -0.8 -2.6 270) (size 0.5 2.5) (layers "F.Cu" "F.Paste" "F.Mask")
       (net 2 "/D-") (pinfunction "D-") (pintype "bidirectional"))
-    (pad "3" smd rect (at 0 -2.6 270) (size 0.5 2.5) (layers "F.Cu" "F.Paste" "F.Mask")
+    (pad "3" smd rect locked (at 0 -2.6 270) (size 0.5 2.5) (layers "F.Cu" "F.Paste" "F.Mask")
       (net 3 "/D+") (pinfunction "D+") (pintype "bidirectional"))
-    (pad "4" smd rect (at 0.8 -2.6 270) (size 0.5 2.5) (layers "F.Cu" "F.Paste" "F.Mask")
+    (pad "4" smd rect locked (at 0.8 -2.6 270) (size 0.5 2.5) (layers "F.Cu" "F.Paste" "F.Mask")
       (net 4 "unconnected-(J1-Pad4)") (pinfunction "ID") (pintype "passive"))
-    (pad "5" smd rect (at 1.6 -2.6 270) (size 0.5 2.5) (layers "F.Cu" "F.Paste" "F.Mask")
+    (pad "5" smd rect locked (at 1.6 -2.6 270) (size 0.5 2.5) (layers "F.Cu" "F.Paste" "F.Mask")
       (net 18 "GND") (pinfunction "GND") (pintype "power_out"))
-    (pad "6" smd rect (at 4.4 2.9 270) (size 2 2.5) (layers "F.Cu" "F.Paste" "F.Mask")
+    (pad "6" smd rect locked (at 4.4 2.9 270) (size 2 2.5) (layers "F.Cu" "F.Paste" "F.Mask")
       (net 18 "GND") (pinfunction "Shield") (pintype "passive"))
-    (pad "6" smd rect (at -4.4 2.9 270) (size 2 2.5) (layers "F.Cu" "F.Paste" "F.Mask")
+    (pad "6" smd rect locked (at -4.4 2.9 270) (size 2 2.5) (layers "F.Cu" "F.Paste" "F.Mask")
       (net 18 "GND") (pinfunction "Shield") (pintype "passive"))
-    (pad "6" smd rect (at 4.4 -2.6 270) (size 2 2.5) (layers "F.Cu" "F.Paste" "F.Mask")
+    (pad "6" smd rect locked (at 4.4 -2.6 270) (size 2 2.5) (layers "F.Cu" "F.Paste" "F.Mask")
       (net 18 "GND") (pinfunction "Shield") (pintype "passive"))
-    (pad "6" smd rect (at -4.4 -2.6 270) (size 2 2.5) (layers "F.Cu" "F.Paste" "F.Mask")
+    (pad "6" smd rect locked (at -4.4 -2.6 270) (size 2 2.5) (layers "F.Cu" "F.Paste" "F.Mask")
       (net 18 "GND") (pinfunction "Shield") (pintype "passive"))
-    (pad "GND" thru_hole circle (at 5.08 5.08 270) (size 1 1) (drill 0.5) (layers *.Cu *.Mask))
-    (pad "GND" thru_hole circle (at -5.08 5.08 270) (size 1 1) (drill 0.5) (layers *.Cu *.Mask))
-    (pad "GND" thru_hole circle (at 5.08 0 270) (size 1 1) (drill 0.5) (layers *.Cu *.Mask))
-    (pad "GND" thru_hole circle (at -5.08 0 270) (size 1 1) (drill 0.5) (layers *.Cu *.Mask))
+    (pad "GND" thru_hole circle locked (at 5.08 5.08 270) (size 1 1) (drill 0.5) (layers *.Cu *.Mask))
+    (pad "GND" thru_hole circle locked (at -5.08 5.08 270) (size 1 1) (drill 0.5) (layers *.Cu *.Mask))
+    (pad "GND" thru_hole circle locked (at 5.08 0 270) (size 1 1) (drill 0.5) (layers *.Cu *.Mask))
+    (pad "GND" thru_hole circle locked (at -5.08 0 270) (size 1 1) (drill 0.5) (layers *.Cu *.Mask))
     (model "${KICAD6_3DMODEL_DIR}/Connector_USB.3dshapes/USB_Mini-B_Wuerth_65100516121_Horizontal.wrl"
       (offset (xyz 0 0 0))
@@
     )
   )
-  (gr_rect (start 127 101.6) (end 177.8 76.2) (layer "Edge.Cuts") (width 0.1) (fill none))
+  (gr_line (start 127 100.33) (end 127 93.98) (layer "Edge.Cuts") (width 0.1))
+  (gr_line (start 127 83.82) (end 127 77.47) (layer "Edge.Cuts") (width 0.1))
+  (gr_line (start 127 77.47) (end 128.27 76.2) (layer "Edge.Cuts") (width 0.1))
+  (gr_line (start 176.53 101.6) (end 177.8 100.33) (layer "Edge.Cuts") (width 0.1))
+  (gr_line (start 127 100.33) (end 128.27 101.6) (layer "Edge.Cuts") (width 0.1))
+  (gr_line (start 127 93.98) (end 128.27 92.71) (layer "Edge.Cuts") (width 0.1))
+  (gr_line (start 177.8 77.47) (end 177.8 100.33) (layer "Edge.Cuts") (width 0.1))
+  (gr_line (start 128.27 92.71) (end 128.27 85.09) (layer "Edge.Cuts") (width 0.1))
+  (gr_line (start 128.27 76.2) (end 176.53 76.2) (layer "Edge.Cuts") (width 0.1))
+  (gr_line (start 176.53 76.2) (end 177.8 77.47) (layer "Edge.Cuts") (width 0.1))
+  (gr_line (start 128.27 85.09) (end 127 83.82) (layer "Edge.Cuts") (width 0.1))
+  (gr_line (start 176.53 101.6) (end 128.27 101.6) (layer "Edge.Cuts") (width 0.1))
   (segment (start 154.305 92.645) (end 154.1262 91.6751) (width 0.5) (layer "F.Cu") (net 2))
   (segment (start 152.6078 89.9184) (end 139.6447 89.9184) (width 0.5) (layer "F.Cu") (net 2))

Commit message: Signed-off-by: Dmitry Ponyatov <dponyatov@gmail.com>
Parts:
- added C1: 10uF, smd:C_0805, F.Cu at (140.3, 85.5)
- added C2: 10uF, smd:C_0805, F.Cu at (141.0, 82.2)
- added J2: Conn_01x03, connector:PinHeader_1x03_P2.54mm_Vertical, F.Cu at (144.8, 88.9)
- added J3: Conn_01x08, Connector_PinHeader_2.54mm:PinHeader_1x08_P2.54mm_Horizontal, B.Cu at (171.7, 83.1)
- added J4: Conn_01x04_Male, Connector_PinHeader_2.54mm:PinHeader_1x04_P2.54mm_Horizontal, B.Cu at (170.6, 96.8)
- added U2: AMS1117-3.3, Package_TO_SOT_SMD:SOT-223-3_TabPin2, F.Cu at (146.7, 83.2)
- J1: value USB_B_Mini -> M-1J
- moved U1 5.47 mm to (155.1, 95.0)
- moved J1 1.27 mm to (133.3, 88.9)
Connections:
- U1 pad 10: unconnected-(U1-Pad10) -> /DSR
- U1 pad 11: unconnected-(U1-Pad11) -> /RI
- U1 pad 12: unconnected-(U1-Pad12) -> /DCD
- U1 pad 13: unconnected-(U1-Pad13) -> /DTR
- U1 pad 14: unconnected-(U1-Pad14) -> /RTS
- U1 pad 16: unconnected-(U1-Pad16) -> /VCCIO
- U1 pad 2: unconnected-(U1-Pad2) -> /TxD
- U1 pad 3: unconnected-(U1-Pad3) -> /RxD
- U1 pad 9: unconnected-(U1-Pad9) -> /CTS
Routing:
- net /VCCIO: track 0.00 -> 32.3 mm, vias 0 -> 2
- net /TxD: track 0.00 -> 23.5 mm
- net /RxD: track 0.00 -> 22.0 mm
- net /VCC3: track 0.00 -> 18.0 mm
- net /CTS: track 0.00 -> 14.6 mm
- net /DSR: track 0.00 -> 14.2 mm
- net VCC5: track 0.00 -> 13.8 mm
- net /RI: track 0.00 -> 13.2 mm
- net /DCD: track 0.00 -> 12.1 mm
- net /DTR: track 0.00 -> 11.9 mm
- net /RTS: track 0.00 -> 11.2 mm
- net /D-: track 20.8 -> 25.8 mm
- net /D+: track 19.1 -> 23.9 mm
- net GND: track 35.5 -> 34.3 mm, vias 0 -> 1
- added copper zone on B.Cu, net GND
Other:
- outline, holes or cut-outs redrawn
