File: pcb/pwm/pwm.kicad_pcb (KiCad board)
At the start: 2 copper layers, 8 parts, among them Q1 IRFB4321PBF, Q2 IRFB4321PBF, Q3 IRFB4321PBF, Q4 IRFB4321PBF, Q5 IRFB4321PBF, Q6 IRFB4321PBF, Q7 IRFB4321PBF, Q8 IRFB4321PBF

Commit message: Signed-off-by: Dmitry Ponyatov <dponyatov@samsa.local>
Parts:
- added REF**: RQD6010MS, fan:RQD6010MS, F.Cu at (132.1, 40.6)
- added REF**: RQD6010MS, fan:RQD6010MS, F.Cu at (58.4, 40.6)
- moved Q7 61.4 mm to (147.3, 104.1), turned to 90 degrees
- moved Q8 59.1 mm to (147.3, 129.5), turned to 90 degrees
- moved Q5 51.6 mm to (152.4, 66.0), turned to 90 degrees
- moved Q6 36.9 mm to (149.9, 83.8), turned to 90 degrees
- moved Q3 8.03 mm to (76.2, 101.6)
Other:
- board outline added: 154.9 x 152.4 mm

Commit message: Signed-off-by: Dmitry Ponyatov <dponyatov@gmail.com>
Parts:
- added REF**: pwm_radiator, radiator:pwm_radiator, F.Cu at (134.6, 96.5)
- added REF**: pwm_radiator, radiator:pwm_radiator, F.Cu at (55.9, 99.1)
- moved Q4 26.9 mm to (50.8, 133.3)
- moved Q1 26.7 mm to (50.8, 59.7)
- moved Q3 26.6 mm to (51.1, 110.5)
- moved Q2 25.9 mm to (50.8, 83.8)
- moved Q7 13.9 mm to (139.4, 115.6)
- moved Q5 12.8 mm to (139.7, 64.3)
- moved Q8 11.9 mm to (139.4, 138.4)
- moved Q6 11.4 mm to (139.7, 88.9)
Changed lines of the file:
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@@
   (net 11 "Net-(Q8-Pad1)")
   (footprint "Package_TO_SOT_THT:TO-220-3_Vertical" (layer "F.Cu")
-    (at 147.32 129.54 90)
+    (at 139.375 138.43 90)
     (descr "TO-220-3, Vertical, RM 2.54mm, see https://www.vishay.com/docs/66542/to-220-1.pdf")
     (tags "TO-220-3 Vertical RM 2.54mm")
@@
   )
   (footprint "Package_TO_SOT_THT:TO-220-3_Vertical" (layer "F.Cu")
-    (at 149.86 83.82 90)
+    (at 139.7 88.9 90)
     (descr "TO-220-3, Vertical, RM 2.54mm, see https://www.vishay.com/docs/66542/to-220-1.pdf")
     (tags "TO-220-3 Vertical RM 2.54mm")
@@
   )
   (footprint "Package_TO_SOT_THT:TO-220-3_Vertical" (layer "F.Cu")
-    (at 77.49 60.96 -90)
+    (at 50.8 59.69 -90)
     (descr "TO-220-3, Vertical, RM 2.54mm, see https://www.vishay.com/docs/66542/to-220-1.pdf")
     (tags "TO-220-3 Vertical RM 2.54mm")
@@
   )
   (footprint "Package_TO_SOT_THT:TO-220-3_Vertical" (layer "F.Cu")
-    (at 147.32 104.14 90)
+    (at 139.375 115.57 90)
     (descr "TO-220-3, Vertical, RM 2.54mm, see https://www.vishay.com/docs/66542/to-220-1.pdf")
     (tags "TO-220-3 Vertical RM 2.54mm")
@@
   )
   (footprint "Package_TO_SOT_THT:TO-220-3_Vertical" (layer "F.Cu")
-    (at 152.4 66.04 90)
+    (at 139.7 64.269 90)
     (descr "TO-220-3, Vertical, RM 2.54mm, see https://www.vishay.com/docs/66542/to-220-1.pdf")
     (tags "TO-220-3 Vertical RM 2.54mm")
@@
   )
   (footprint "Package_TO_SOT_THT:TO-220-3_Vertical" (layer "F.Cu")
-    (at 76.24 78.74 -90)
+    (at 50.8 83.82 -90)
     (descr "TO-220-3, Vertical, RM 2.54mm, see https://www.vishay.com/docs/66542/to-220-1.pdf")
     (tags "TO-220-3 Vertical RM 2.54mm")
@@
     )
   )
-  (footprint "Package_TO_SOT_THT:TO-220-3_Vertical" (layer "F.Cu")
-    (at 76.2 124.46 -90)
+  (footprint "radiator:pwm_radiator" (layer "F.Cu")
+    (at 134.62 96.52)
+    (fp_text reference "REF**" (at 0 -0.5 unlocked) (layer "F.SilkS")
+      (effects (font (size 1 1) (thickness 0.15)))
+    )
+    (fp_text value "pwm_radiator" (at 0 1 unlocked) (layer "F.Fab")
+      (effects (font (size 1 1) (thickness 0.15)))
+    )
+    (fp_text user "${REFERENCE}" (at 0 2.5 unlocked) (layer "F.Fab")
+      (effects (font (size 1 1) (thickness 0.15)))
+    )
+    (fp_line (start 1 -49) (end 1 51) (layer "Edge.Cuts") (width 0.12))
+    (fp_circle (center -8 -30) (end -6 -30) (layer "Edge.Cuts") (width 0.12) (fill none))
+    (fp_circle (center -9 30) (end -7 30) (layer "Edge.Cuts") (width 0.12) (fill none))
+    (fp_rect (start 1 -51) (end -19 54) (layer "F.CrtYd") (width 0.12) (fill none))
+    (fp_rect (start -16 -49) (end 15 51) (layer "F.Fab") (width 0.12) (fill none))
+  )
+  (footprint "Package_TO_SOT_THT:TO-220-3_Vertical" (layer "F.Cu")
+    (at 50.8 133.35 -90)
     (descr "TO-220-3, Vertical, RM 2.54mm, see https://www.vishay.com/docs/66542/to-220-1.pdf")
     (tags "TO-220-3 Vertical RM 2.54mm")
@@
     )
   )
-  (footprint "Package_TO_SOT_THT:TO-220-3_Vertical" (layer "F.Cu")
-    (at 76.2 101.6 -90)
-    (descr "TO-220-3, Vertical, RM 2.54mm, see https://www.vishay.com/docs/66542/to-220-1.pdf")
-    (tags "TO-220-3 Vertical RM 2.54mm")
+  (footprint "radiator:pwm_radiator" (layer "F.Cu")
+    (at 55.88 99.06 180)
+    (fp_text reference "REF**" (at 0 -0.5 180 unlocked) (layer "F.SilkS")
+      (effects (font (size 1 1) (thickness 0.15)))
+    )
+    (fp_text value "pwm_radiator" (at 0 1 180 unlocked) (layer "F.Fab")
+      (effects (font (size 1 1) (thickness 0.15)))
+    )
+    (fp_text user "${REFERENCE}" (at 0 2.5 180 unlocked) (layer "F.Fab")
+      (effects (font (size 1 1) (thickness 0.15)))
+    )
+    (fp_line (start 1 -49) (end 1 51) (layer "Edge.Cuts") (width 0.12))
+    (fp_circle (center -9 30) (end -7 30) (layer "Edge.Cuts") (width 0.12) (fill none))
+    (fp_circle (center -8 -30) (end -6 -30) (layer "Edge.Cuts") (width 0.12) (fill none))
+    (fp_rect (start 1 -51) (end -19 54) (layer "F.CrtYd") (width 0.12) (fill none))
+    (fp_rect (start -16 -49) (end 15 51) (layer "F.Fab") (width 0.12) (fill none))
+  )
+  (footprint "Package_TO_SOT_THT:TO-220-3_Vertical" (layer "F.Cu")
+    (at 51.125 110.49 -90)
+    (descr "TO-220-3, Vertical, RM 2.54mm, see https://www.vishay.com/docs/66542/to-220-1.pdf")
+    (tags "TO-220-3 Vertical RM 2.54mm")

Commit message: Signed-off-by: Dmitry Ponyatov <dponyatov@samsa.local>
Parts:
- added U1: pwm_meson0, pwm_meson:pwm_meson0, F.Cu at (95.2, 106.7)
- added X1: Conn_01x04_Male, terminal:PLS-4, F.Cu at (106.7, 147.3)
- added X2: Conn_01x04_Male, terminal:PLS-4, F.Cu at (83.8, 147.3)
- added X3: Conn_01x02_Male, terminal:CWF-2, F.Cu at (101.6, 62.5)
- added X4: Fan, terminal:CWF-2, F.Cu at (86.4, 62.5)
- moved REF** 2.84 mm to (55.9, 39.4)
- moved Q5 2.83 mm to (139.2, 67.1)
- moved REF** 1.27 mm to (132.1, 39.4)
Connections:
- net Net-(Q5-Pad1) renamed /G5
- net Net-(Q6-Pad1) renamed /G6
- net Net-(Q7-Pad1) renamed /G7
- net Net-(Q8-Pad1) renamed /G8
Routing:
- net /phase: track 0.00 -> 123.1 mm
- net /+60V: track 0.00 -> 98.6 mm
- net /fan+: track 0.00 -> 85.2 mm
- net /fan-: track 0.00 -> 69.6 mm
Other:
- board size 154.9 x 152.4 mm -> 145 x 145 mm

Commit message: Signed-off-by: Dmitry Ponyatov <dponyatov@samsa.local>
Parts:
- added R1: B57045K, Resistor_THT:R_Axial_DIN0411_L9.9mm_D3.6mm_P7.62mm_Vertical, F.Cu at (76.2, 89.9)
- added R2: B57045K, Resistor_THT:R_Axial_DIN0411_L9.9mm_D3.6mm_P7.62mm_Vertical, F.Cu at (114.3, 89.9)
- X4: value Fan -> Conn_01x02_Male
- moved Q4 4.87 mm to (51.4, 128.5)
- moved Q3 3.98 mm to (51.4, 106.5)
- moved Q1 2.90 mm to (51.4, 62.5)
- moved Q2 0.95 mm to (51.4, 84.5)
Connections:
- U1 pad 5A: (no net) -> /t1-
- U1 pad 5J: (no net) -> /t2-
- U1 pad 7A: (no net) -> /t1+
- U1 pad 7J: (no net) -> /t2+
Routing:
- net /+60V: track 98.6 -> 0.00 mm
- net /phase: track 123.1 -> 26.1 mm
- net /t2-: track 0.00 -> 8.80 mm
- net /t1-: track 0.00 -> 8.67 mm
- net /t2+: track 0.00 -> 7.74 mm
- net /t1+: track 0.00 -> 7.74 mm
- net /-60V: track 0.00 -> 4.95 mm
- added copper zone on B.Cu, net /+60V
- added copper zone on B.Cu, net /-60V
- added copper zone on B.Cu, net /phase

Commit message: Signed-off-by: Dmitry Ponyatov <dponyatov@gmail.com>
Routing:
- net /+60V: track 0.00 -> 18.9 mm
- net /-60V: track 4.95 -> 21.1 mm
- net /phase: track 26.1 -> 28.5 mm
Changed lines of the file:
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@@
   )
   (gr_rect (start 21.37 29.21) (end 166.37 174.21) (layer "Edge.Cuts") (width 0.1) (fill none))
-  (segment (start 139.7 86.36) (end 137.16 86.36) (width 1.27) (layer "B.Cu") (net 3))
-  (segment (start 51.435 89.6) (end 55.31 89.6) (width 1.27) (layer "B.Cu") (net 3))
-  (segment (start 51.630407 111.76) (end 55.88 111.76) (width 1.27) (layer "B.Cu") (net 3))
+  (segment (start 51.435 131.06) (end 48.01 131.06) (width 1.27) (layer "B.Cu") (net 2))
+  (segment (start 47.56 87.06) (end 46.99 87.63) (width 1.27) (layer "B.Cu") (net 2))
+  (segment (start 51.435 87.06) (end 47.56 87.06) (width 1.27) (layer "B.Cu") (net 2))
+  (segment (start 47.15 109.06) (end 46.99 109.22) (width 1.27) (layer "B.Cu") (net 2))
+  (segment (start 51.435 65.06) (end 47.97 65.06) (width 1.27) (layer "B.Cu") (net 2))
+  (segment (start 51.435 109.06) (end 47.15 109.06) (width 1.27) (layer "B.Cu") (net 2))
+  (segment (start 47.97 65.06) (end 46.99 66.04) (width 1.27) (layer "B.Cu") (net 2))
+  (segment (start 48.01 131.06) (end 46.99 132.08) (width 1.27) (layer "B.Cu") (net 2))
+  (segment (start 54.36 133.6) (end 54.61 133.35) (width 1.27) (layer "B.Cu") (net 3))
+  (segment (start 51.435 67.6) (end 54.32 67.6) (width 1.27) (layer "B.Cu") (net 3))
   (segment (start 51.435 111.6) (end 51.470407 111.6) (width 1.27) (layer "B.Cu") (net 3))
-  (segment (start 51.435 67.6) (end 54.9 67.6) (width 1.27) (layer "B.Cu") (net 3))
-  (segment (start 54.9 67.6) (end 55.88 68.58) (width 1.27) (layer "B.Cu") (net 3))
+  (segment (start 139.375 113.03) (end 135.89 113.03) (width 1.27) (layer "B.Cu") (net 3))
+  (segment (start 51.435 111.6) (end 53.5 111.6) (width 1.27) (layer "B.Cu") (net 3))
+  (segment (start 51.435 133.6) (end 54.36 133.6) (width 1.27) (layer "B.Cu") (net 3))
+  (segment (start 135.89 64.77) (end 136.144 64.516) (width 1.27) (layer "B.Cu") (net 3))
+  (segment (start 53.91 89.6) (end 54.61 88.9) (width 1.27) (layer "B.Cu") (net 3))
   (segment (start 139.192 64.516) (end 139.156593 64.516) (width 1.27) (layer "B.Cu") (net 3))
-  (segment (start 55.31 89.6) (end 55.88 90.17) (width 1.27) (layer "B.Cu") (net 3))
-  (segment (start 139.192 64.516) (end 134.62 64.516) (width 1.27) (layer "B.Cu") (net 3))
-  (segment (start 55.88 133.35) (end 55.63 133.6) (width 1.27) (layer "B.Cu") (net 3))
+  (segment (start 139.375 135.89) (end 135.89 135.89) (width 1.27) (layer "B.Cu") (net 3))
+  (segment (start 139.192 64.516) (end 136.144 64.516) (width 1.27) (layer "B.Cu") (net 3))
   (segment (start 139.156593 64.516) (end 138.902593 64.77) (width 1.27) (layer "B.Cu") (net 3))
-  (segment (start 51.435 133.6) (end 55.63 133.6) (width 1.27) (layer "B.Cu") (net 3))
+  (segment (start 53.5 111.6) (end 54.61 110.49) (width 1.27) (layer "B.Cu") (net 3))
+  (segment (start 54.61 67.31) (end 54.32 67.6) (width 1.27) (layer "B.Cu") (net 3))
+  (segment (start 139.7 86.36) (end 135.89 86.36) (width 1.27) (layer "B.Cu") (net 3))
+  (segment (start 51.435 89.6) (end 53.91 89.6) (width 1.27) (layer "B.Cu") (net 3))
   (segment (start 51.470407 111.6) (end 51.630407 111.76) (width 1.27) (layer "B.Cu") (net 3))
-  (segment (start 139.192 61.976) (end 141.986 61.976) (width 1.27) (layer "B.Cu") (net 7))
-  (segment (start 141.986 61.976) (end 143.51 63.5) (width 1.27) (layer "B.Cu") (net 7))
+  (segment (start 139.192 61.976) (end 143.256 61.976) (width 1.27) (layer "B.Cu") (net 7))
+  (segment (start 139.7 83.82) (end 143.51 83.82) (width 1.27) (layer "B.Cu") (net 7))
+  (segment (start 139.375 110.49) (end 143.51 110.49) (width 1.27) (layer "B.Cu") (net 7))
+  (segment (start 139.375 109.545) (end 142.24 106.68) (width 1.27) (layer "B.Cu") (net 7))
+  (segment (start 139.375 133.35) (end 143.51 133.35) (width 1.27) (layer "B.Cu") (net 7))
+  (segment (start 139.375 110.49) (end 139.375 109.545) (width 1.27) (layer "B.Cu") (net 7))
   (segment (start 95.504 104.394) (end 95.504 63.754) (width 1.27) (layer "B.Cu") (net 8))
   (segment (start 95.504 63.754) (end 91.694 63.754) (width 1.27) (layer "B.Cu") (net 8))
@@
   (segment (start 106.68 85.09) (end 111.46 85.09) (width 1.27) (layer "B.Cu") (net 25))
   (segment (start 111.46 85.09) (end 114.3 82.25) (width 1.27) (layer "B.Cu") (net 25))
-  (zone (net 3) (net_name "/phase") (layer "B.Cu") (name "phase") (hatch edge 0.508)
+  (zone (net 3) (net_name "/phase") (layer "B.Cu") (hatch edge 0.508)
     (connect_pads (clearance 2))
-    (min_thickness 2.54) (filled_areas_thickness no)
-    (fill yes (thermal_gap 2.54) (thermal_bridge_width 2.54) (smoothing fillet) (radius 2) (island_removal_mode 1) (island_area_min 0))
+    (min_thickness 0.254) (filled_areas_thickness no)
+    (fill yes (thermal_gap 0.254) (thermal_bridge_width 0.254) (smoothing fillet) (radius 5))
     (polygon
       (pts
-        (xy 72.39 152.4)
-        (xy 53.34 152.4)
-        (xy 53.34 58.42)
-        (xy 72.39 58.42)
-      )
-    )
-  )
-  (zone (net 3) (net_name "/phase") (layer "B.Cu") (name "phase") (hatch edge 0.508)
-    (connect_pads (clearance 2))
-    (min_thickness 1.27) (filled_areas_thickness no)
-    (fill yes (thermal_gap 2.54) (thermal_bridge_width 1.27) (smoothing fillet) (radius 5))
-    (polygon
-      (pts
-        (xy 137.16 149.86)
         (xy 118.11 152.4)
         (xy 118.11 58.42)
         (xy 137.16 58.42)
+        (xy 135.89 154.94)
+        (xy 114.3 170.18)
+        (xy 76.2 170.18)
+        (xy 53.34 154.94)
+        (xy 53.34 58.42)
+        (xy 72.39 58.42)
+        (xy 72.39 152.4)
       )
     )
@@
   )
   (zone (net 7) (net_name "/-60V") (layer "B.Cu") (name "+60V") (hatch edge 0.508)
-    (connect_pads (clearance 2))
+    (connect_pads (clearance 2.54))
     (min_thickness 2.54) (filled_areas_thickness no)
     (fill yes (thermal_gap 2.54) (thermal_bridge_width 2.54) (smoothing fillet) (radius 5) (island_removal_mode 1) (island_area_min 0))
@@
         (xy 139.7 160.02)
         (xy 142.24 154.94)
-        (xy 142.24 58.42)
+        (xy 140.97 58.42)
         (xy 160.02 58.42)
       )
     )
-  )
-  (zone (net 3) (net_name "/phase") (layer "B.Cu") (name "phase") (hatch edge 0.508)
-    (connect_pads (clearance 2))
-    (min_thickness 2.54) (filled_areas_thickness no)
-    (fill yes (thermal_gap 2.54) (thermal_bridge_width 2.54) (smoothing fillet) (radius 5) (island_removal_mode 1) (island_area_min 0))
-    (polygon
-      (pts
-        (xy 78.74 152.4)
-        (xy 111.76 152.4)
-        (xy 119.38 149.86)
-        (xy 137.16 149.86)
-        (xy 137.16 154.94)
-        (xy 114.3 160.02)
-        (xy 114.3 170.18)
-        (xy 76.2 170.18)
-        (xy 76.2 160.02)
-        (xy 53.34 154.94)
-        (xy 53.34 149.86)
-        (xy 71.12 149.86)
-      )
-    )
