File: pcb/pwm/pwm.kicad_pcb (KiCad board)
At the start: 2 copper layers, 145 x 145 mm, 19 parts, among them Q1 IRFB4321PBF, Q2 IRFB4321PBF, Q3 IRFB4321PBF, Q4 IRFB4321PBF, Q5 IRFB4321PBF, Q6 IRFB4321PBF, Q7 IRFB4321PBF, Q8 IRFB4321PBF, U1 pwm_meson0, X1 Conn_01x04_Male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

Commit message: Signed-off-by: Dmitry Ponyatov <dponyatov@samsa.local>
Parts:
- Q1, Q2, Q3, Q4, Q5, Q6, Q7, Q8: footprint Package_TO_SOT_THT:TO-220-3_Vertical -> mosfet:TO-220AB
Routing:
- net /+60V: track 18.9 -> 51.8 mm
- net /phase: track 28.5 -> 54.1 mm
- net /-60V: track 21.1 -> 37.3 mm

Commit message: Signed-off-by: Dmitry Ponyatov <dponyatov@samsa.local>
Parts:
- Q1, Q2, Q3, Q4, Q5, Q6, Q7, Q8: footprint mosfet:TO-220AB -> Package_TO_SOT_THT:TO-220-3_Vertical
- moved X1 2.54 mm to (104.1, 147.3)
- moved X2 2.54 mm to (86.4, 147.3)
Connections:
- U1 pad 20J: (no net) -> /+12V
- U1 pad 22J: (no net) -> /-12V
Routing:
- net /+12V: track 0.00 -> 31.8 mm
- net /-12V: track 0.00 -> 24.2 mm

Commit message: Signed-off-by: Dmitry Ponyatov <dponyatov@samsa.local>
Connections:
- U1 pad 16A: (no net) -> /+24V
- U1 pad 16J: (no net) -> /-24V
Routing:
- net /-24V: track 0.00 -> 45.9 mm
- net /+24V: track 0.00 -> 40.5 mm
Changed lines of the file:
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@@
     (pad "15A" thru_hole oval (at -11.43 3.81) (size 3 1.524) (drill 0.762) (layers *.Cu *.Mask))
     (pad "15J" thru_hole oval (at 11.43 3.81) (size 3 1.524) (drill 0.762) (layers *.Cu *.Mask))
-    (pad "16A" thru_hole oval (at -11.43 6.35) (size 3 1.524) (drill 0.762) (layers *.Cu *.Mask))
-    (pad "16J" thru_hole oval (at 11.43 6.35) (size 3 1.524) (drill 0.762) (layers *.Cu *.Mask))
+    (pad "16A" thru_hole oval (at -11.43 6.35) (size 3 1.524) (drill 0.762) (layers *.Cu *.Mask)
+      (net 18 "/+24V") (pinfunction "+24V") (pintype "power_out"))
+    (pad "16J" thru_hole oval (at 11.43 6.35) (size 3 1.524) (drill 0.762) (layers *.Cu *.Mask)
+      (net 20 "/-24V") (pinfunction "-24V") (pintype "power_out"))
     (pad "17A" thru_hole oval (at -11.43 8.89) (size 3 1.524) (drill 0.762) (layers *.Cu *.Mask))
     (pad "17J" thru_hole oval (at 11.43 8.89) (size 3 1.524) (drill 0.762) (layers *.Cu *.Mask))
@@
   (segment (start 104.14 128.27) (end 106.68 128.27) (width 1.27) (layer "B.Cu") (net 16))
   (segment (start 105.41 143.51) (end 101.6 139.7) (width 1.27) (layer "B.Cu") (net 16))
+  (segment (start 82.55 142.24) (end 88.9 135.89) (width 1.27) (layer "B.Cu") (net 18))
+  (segment (start 82.55 147.32) (end 82.55 142.24) (width 1.27) (layer "B.Cu") (net 18))
+  (segment (start 88.9 115.57) (end 86.36 113.03) (width 1.27) (layer "B.Cu") (net 18))
+  (segment (start 86.36 113.03) (end 83.82 113.03) (width 1.27) (layer "B.Cu") (net 18))
+  (segment (start 88.9 135.89) (end 88.9 115.57) (width 1.27) (layer "B.Cu") (net 18))
+  (segment (start 100.33 113.03) (end 106.68 113.03) (width 1.27) (layer "B.Cu") (net 20))
+  (segment (start 92.71 120.65) (end 100.33 113.03) (width 1.27) (layer "B.Cu") (net 20))
+  (segment (start 87.63 147.32) (end 87.63 144.78) (width 1.27) (layer "B.Cu") (net 20))
+  (segment (start 87.63 144.78) (end 92.71 139.7) (width 1.27) (layer "B.Cu") (net 20))
+  (segment (start 92.71 139.7) (end 92.71 120.65) (width 1.27) (layer "B.Cu") (net 20))
   (segment (start 76.5 90.17) (end 76.2 89.87) (width 1.27) (layer "B.Cu") (net 22))
   (segment (start 83.82 90.17) (end 76.5 90.17) (width 1.27) (layer "B.Cu") (net 22))

Commit message: Signed-off-by: Dmitry Ponyatov <dponyatov@samsa.local>
Parts:
- moved R1 1.98 mm to (76.2, 91.8)
Connections:
- U1 pad 10A: (no net) -> /+60V
- U1 pad 12A: (no net) -> /G3
- U1 pad 1A: (no net) -> /G1
- U1 pad 20A: (no net) -> /G4
- U1 pad 3A: (no net) -> /G2
Routing:
- net /G1: track 0.00 -> 43.6 mm
- net /G2: track 0.00 -> 41.4 mm
- net /+60V: track 51.8 -> 87.4 mm
- net /t1-: track 8.67 -> 7.98 mm
- net /t1+: track 7.74 -> 8.32 mm
- net (no net): vias 0 -> 4
Changed lines of the file:
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@@
   )
   (footprint "Resistor_THT:R_Axial_DIN0411_L9.9mm_D3.6mm_P7.62mm_Vertical" (layer "F.Cu")
-    (at 76.2 89.87 90)
+    (at 76.2 91.85 90)
     (descr "Resistor, Axial_DIN0411 series, Axial, Vertical, pin pitch=7.62mm, 1W, length*diameter=9.9*3.6mm^2")
     (tags "Resistor Axial_DIN0411 series Axial Vertical pin pitch 7.62mm 1W length 9.9mm diameter 3.6mm")
@@
     (fp_circle (center 12.5 30.5) (end 13.5 30.5) (layer "Edge.Cuts") (width 0.12) (fill none))
     (fp_rect (start -17 -39) (end 17 35) (layer "F.CrtYd") (width 0.05) (fill none))
-    (pad "1A" thru_hole rect (at -11.43 -31.75) (size 3 1.524) (drill 0.762) (layers *.Cu *.Mask))
+    (pad "1A" thru_hole rect (at -11.43 -31.75) (size 3 1.524) (drill 0.762) (layers *.Cu *.Mask)
+      (net 1 "/G1") (pinfunction "Q1") (pintype "output"))
     (pad "1J" thru_hole oval (at 11.43 -31.75) (size 3 1.524) (drill 0.762) (layers *.Cu *.Mask))
     (pad "2A" thru_hole oval (at -11.43 -29.21) (size 3 1.524) (drill 0.762) (layers *.Cu *.Mask))
     (pad "2J" thru_hole oval (at 11.43 -29.21) (size 3 1.524) (drill 0.762) (layers *.Cu *.Mask))
-    (pad "3A" thru_hole oval (at -11.43 -26.67) (size 3 1.524) (drill 0.762) (layers *.Cu *.Mask))
+    (pad "3A" thru_hole oval (at -11.43 -26.67) (size 3 1.524) (drill 0.762) (layers *.Cu *.Mask)
+      (net 4 "/G2") (pinfunction "Q2") (pintype "output"))
     (pad "3J" thru_hole oval (at 11.43 -26.67) (size 3 1.524) (drill 0.762) (layers *.Cu *.Mask))
     (pad "4A" thru_hole oval (at -11.43 -24.13) (size 3 1.524) (drill 0.762) (layers *.Cu *.Mask))
@@
     (pad "9A" thru_hole oval (at -11.43 -11.43) (size 3 1.524) (drill 0.762) (layers *.Cu *.Mask))
     (pad "9J" thru_hole oval (at 11.43 -11.43) (size 3 1.524) (drill 0.762) (layers *.Cu *.Mask))
-    (pad "10A" thru_hole oval (at -11.43 -8.89) (size 3 1.524) (drill 0.762) (layers *.Cu *.Mask))
+    (pad "10A" thru_hole oval (at -11.43 -8.89) (size 3 1.524) (drill 0.762) (layers *.Cu *.Mask)
+      (net 2 "/+60V") (pinfunction "+60V") (pintype "power_out"))
     (pad "10J" thru_hole oval (at 11.43 -8.89) (size 3 1.524) (drill 0.762) (layers *.Cu *.Mask))
     (pad "11A" thru_hole oval (at -11.43 -6.35) (size 3 1.524) (drill 0.762) (layers *.Cu *.Mask))
     (pad "11J" thru_hole oval (at 11.43 -6.35) (size 3 1.524) (drill 0.762) (layers *.Cu *.Mask))
-    (pad "12A" thru_hole oval (at -11.43 -3.81) (size 3 1.524) (drill 0.762) (layers *.Cu *.Mask))
+    (pad "12A" thru_hole oval (at -11.43 -3.81) (size 3 1.524) (drill 0.762) (layers *.Cu *.Mask)
+      (net 5 "/G3") (pinfunction "Q3") (pintype "output"))
     (pad "12J" thru_hole oval (at 11.43 -3.81) (size 3 1.524) (drill 0.762) (layers *.Cu *.Mask))
     (pad "13A" thru_hole oval (at -11.43 -1.27) (size 3 1.524) (drill 0.762) (layers *.Cu *.Mask))
@@
     (pad "19A" thru_hole oval (at -11.43 13.97) (size 3 1.524) (drill 0.762) (layers *.Cu *.Mask))
     (pad "19J" thru_hole oval (at 11.43 13.97) (size 3 1.524) (drill 0.762) (layers *.Cu *.Mask))
-    (pad "20A" thru_hole oval (at -11.43 16.51) (size 3 1.524) (drill 0.762) (layers *.Cu *.Mask))
+    (pad "20A" thru_hole oval (at -11.43 16.51) (size 3 1.524) (drill 0.762) (layers *.Cu *.Mask)
+      (net 6 "/G4") (pinfunction "Q4") (pintype "output"))
     (pad "20J" thru_hole oval (at 11.43 16.51) (size 3 1.524) (drill 0.762) (layers *.Cu *.Mask)
       (net 14 "/+12V") (pinfunction "+12V") (pintype "power_out"))
@@
   )
   (gr_rect (start 21.37 29.21) (end 166.37 174.21) (layer "Edge.Cuts") (width 0.1) (fill none))
+  (via (at 76.2 77.47) (size 2) (drill 0.7) (layers "F.Cu" "B.Cu") (free) (net 0))
+  (via (at 50.8 77.47) (size 2) (drill 0.7) (layers "F.Cu" "B.Cu") (free) (net 0))
+  (via (at 76.2 97.79) (size 2) (drill 0.7) (layers "F.Cu" "B.Cu") (free) (net 0))
+  (via (at 49.53 97.79) (size 2) (drill 0.7) (layers "F.Cu" "B.Cu") (free) (net 0))
+  (segment (start 83.82 74.93) (end 80.01 74.93) (width 1.27) (layer "B.Cu") (net 1))
+  (segment (start 54.265 59.69) (end 51.435 62.52) (width 1.27) (layer "B.Cu") (net 1))
+  (segment (start 80.01 74.93) (end 76.2 71.12) (width 1.27) (layer "B.Cu") (net 1))
+  (segment (start 71.12 59.69) (end 54.265 59.69) (width 1.27) (layer "B.Cu") (net 1))
+  (segment (start 76.2 64.77) (end 71.12 59.69) (width 1.27) (layer "B.Cu") (net 1))
+  (segment (start 76.2 71.12) (end 76.2 64.77) (width 1.27) (layer "B.Cu") (net 1))
+  (segment (start 76.2 97.79) (end 49.53 97.79) (width 1.27) (layer "F.Cu") (net 2))
   (segment (start 50.165 131.06) (end 49.78 131.06) (width 1.27) (layer "B.Cu") (net 2))
   (segment (start 50.165 109.06) (end 49.37 109.06) (width 1.27) (layer "B.Cu") (net 2))
@@
   (segment (start 50.1 87.06) (end 46.99 90.17) (width 1.27) (layer "B.Cu") (net 2))
   (segment (start 50.165 131.06) (end 49.28 131.06) (width 1.27) (layer "B.Cu") (net 2))
+  (segment (start 83.82 97.79) (end 76.2 97.79) (width 1.27) (layer "B.Cu") (net 2))
   (segment (start 49.37 109.06) (end 46.99 106.68) (width 1.27) (layer "B.Cu") (net 2))
+  (segment (start 48.26 97.79) (end 49.53 97.79) (width 1.27) (layer "B.Cu") (net 2))
   (segment (start 50.165 87.06) (end 46.99 83.885) (width 1.27) (layer "B.Cu") (net 2))
   (segment (start 50.165 65.405) (end 46.99 68.58) (width 1.27) (layer "B.Cu") (net 2))
@@
   (segment (start 51.78 67.6) (end 54.61 64.77) (width 1.27) (layer "B.Cu") (net 3))
   (segment (start 51.470407 111.6) (end 51.630407 111.76) (width 1.27) (layer "B.Cu") (net 3))
+  (segment (start 76.2 77.47) (end 50.8 77.47) (width 1.27) (layer "F.Cu") (net 4))
+  (segment (start 51.435 84.52) (end 51.435 78.105) (width 1.27) (layer "B.Cu") (net 4))
+  (segment (start 83.82 80.01) (end 78.74 80.01) (width 1.27) (layer "B.Cu") (net 4))
+  (segment (start 51.435 78.105) (end 50.8 77.47) (width 1.27) (layer "B.Cu") (net 4))
+  (segment (start 78.74 80.01) (end 76.2 77.47) (width 1.27) (layer "B.Cu") (net 4))
   (segment (start 139.192 61.976) (end 139.192 60.198) (width 1.27) (layer "B.Cu") (net 7))
   (segment (start 139.7 83.82) (end 139.7 82.55) (width 1.27) (layer "B.Cu") (net 7))
@@
   (segment (start 87.63 144.78) (end 92.71 139.7) (width 1.27) (layer "B.Cu") (net 20))
   (segment (start 92.71 139.7) (end 92.71 120.65) (width 1.27) (layer "B.Cu") (net 20))
-  (segment (start 76.5 90.17) (end 76.2 89.87) (width 1.27) (layer "B.Cu") (net 22))
-  (segment (start 83.82 90.17) (end 76.5 90.17) (width 1.27) (layer "B.Cu") (net 22))
+  (segment (start 83.82 90.17) (end 77.88 90.17) (width 1.27) (layer "B.Cu") (net 22))
+  (segment (start 77.88 90.17) (end 76.2 91.85) (width 1.27) (layer "B.Cu") (net 22))
   (segment (start 114 90.17) (end 114.3 89.87) (width 1.27) (layer "B.Cu") (net 23))
   (segment (start 106.68 90.17) (end 114 90.17) (width 1.27) (layer "B.Cu") (net 23))
+  (segment (start 76.2 84.23) (end 76.61 84.23) (width 1.27) (layer "B.Cu") (net 24))
+  (segment (start 76.61 84.23) (end 77.47 85.09) (width 1.27) (layer "B.Cu") (net 24))
+  (segment (start 77.47 85.09) (end 78.74 85.09) (width 1.27) (layer "B.Cu") (net 24))
   (segment (start 78.74 85.09) (end 83.82 85.09) (width 1.27) (layer "B.Cu") (net 24))
-  (segment (start 76.2 82.55) (end 78.74 85.09) (width 1.27) (layer "B.Cu") (net 24))
   (segment (start 106.68 85.09) (end 111.46 85.09) (width 1.27) (layer "B.Cu") (net 25))
   (segment (start 111.46 85.09) (end 114.3 82.25) (width 1.27) (layer "B.Cu") (net 25))

Commit message: Signed-off-by: Dmitry Ponyatov <dponyatov@samsa.local>
Routing:
- net /G3: track 0.00 -> 38.7 mm
- net (no net): vias 4 -> 6
Changed lines of the file:
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@@
   )
   (gr_rect (start 21.37 29.21) (end 166.37 174.21) (layer "Edge.Cuts") (width 0.1) (fill none))
+  (via (at 76.2 102.87) (size 2) (drill 0.7) (layers "F.Cu" "B.Cu") (free) (net 0))
   (via (at 76.2 77.47) (size 2) (drill 0.7) (layers "F.Cu" "B.Cu") (free) (net 0))
+  (via (at 50.8 101.6) (size 2) (drill 0.7) (layers "F.Cu" "B.Cu") (free) (net 0))
   (via (at 50.8 77.47) (size 2) (drill 0.7) (layers "F.Cu" "B.Cu") (free) (net 0))
   (via (at 76.2 97.79) (size 2) (drill 0.7) (layers "F.Cu" "B.Cu") (free) (net 0))
@@
   (segment (start 51.435 78.105) (end 50.8 77.47) (width 1.27) (layer "B.Cu") (net 4))
   (segment (start 78.74 80.01) (end 76.2 77.47) (width 1.27) (layer "B.Cu") (net 4))
+  (segment (start 74.93 101.6) (end 50.8 101.6) (width 1.27) (layer "F.Cu") (net 5))
+  (segment (start 76.2 102.87) (end 74.93 101.6) (width 1.27) (layer "F.Cu") (net 5))
+  (segment (start 83.82 102.87) (end 76.2 102.87) (width 1.27) (layer "B.Cu") (net 5))
+  (segment (start 51.435 102.235) (end 50.8 101.6) (width 1.27) (layer "B.Cu") (net 5))
+  (segment (start 51.435 106.52) (end 51.435 102.235) (width 1.27) (layer "B.Cu") (net 5))
   (segment (start 139.192 61.976) (end 139.192 60.198) (width 1.27) (layer "B.Cu") (net 7))
   (segment (start 139.7 83.82) (end 139.7 82.55) (width 1.27) (layer "B.Cu") (net 7))

Commit message: Signed-off-by: Dmitry Ponyatov <dponyatov@samsa.local>
Routing:
- net /G4: track 0.00 -> 38.6 mm
- net (no net): vias 6 -> 8
Changed lines of the file:
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@@
   )
   (gr_rect (start 21.37 29.21) (end 166.37 174.21) (layer "Edge.Cuts") (width 0.1) (fill none))
+  (via (at 50.8 123.19) (size 2) (drill 0.7) (layers "F.Cu" "B.Cu") (free) (net 0))
   (via (at 76.2 102.87) (size 2) (drill 0.7) (layers "F.Cu" "B.Cu") (free) (net 0))
+  (via (at 76.2 123.19) (size 2) (drill 0.7) (layers "F.Cu" "B.Cu") (free) (net 0))
   (via (at 76.2 77.47) (size 2) (drill 0.7) (layers "F.Cu" "B.Cu") (free) (net 0))
   (via (at 50.8 101.6) (size 2) (drill 0.7) (layers "F.Cu" "B.Cu") (free) (net 0))
@@
   (segment (start 51.435 102.235) (end 50.8 101.6) (width 1.27) (layer "B.Cu") (net 5))
   (segment (start 51.435 106.52) (end 51.435 102.235) (width 1.27) (layer "B.Cu") (net 5))
+  (segment (start 76.2 123.19) (end 50.8 123.19) (width 1.27) (layer "F.Cu") (net 6))
+  (segment (start 83.82 123.19) (end 76.2 123.19) (width 1.27) (layer "B.Cu") (net 6))
+  (segment (start 51.435 128.52) (end 51.435 123.825) (width 1.27) (layer "B.Cu") (net 6))
+  (segment (start 51.435 123.825) (end 50.8 123.19) (width 1.27) (layer "B.Cu") (net 6))
   (segment (start 139.192 61.976) (end 139.192 60.198) (width 1.27) (layer "B.Cu") (net 7))
   (segment (start 139.7 83.82) (end 139.7 82.55) (width 1.27) (layer "B.Cu") (net 7))
