File: pcb/pwm/pwm.kicad_sch (KiCad schematic)
At the start: 8 parts, among them Q1 IRFB4321PBF, Q2 IRFB4321PBF, Q3 IRFB4321PBF, Q4 IRFB4321PBF, Q5 IRFB4321PBF, Q6 IRFB4321PBF, Q7 IRFB4321PBF, Q8 IRFB4321PBF

Commit message: Signed-off-by: Dmitry Ponyatov <dponyatov@samsa.local>
Parts:
- added J1: +60V, symbol terminal:Screw_1xM4
- added J2: phase_out, symbol terminal:Screw_1xM4
- added J3: -60V, symbol terminal:Screw_1xM4
- added U1: pwm_meson0, symbol pwm_meson:pwm_meson0
Connections:
- net at Q1.3 (S), Q2.3 (S), Q3.3 (S)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: now also J2.1 (Pin_1), U1. (phase)
- net at Q5.3 (S), Q6.3 (S), Q7.3 (S)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: now also J3.1 (Pin_1), U1. (phase)
- net at Q1.2 (D), Q2.2 (D), Q3.2 (D)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: now also J1.1 (Pin_1), U1. (phase)
Other:
- moved on the sheet: Q5, Q6, Q7, Q8

Commit message: Signed-off-by: Dmitry Ponyatov <dponyatov@samsa.local>
Parts:
- added R1, R2: Thermistor, symbol Device:Thermistor
- added X1, X2: Conn_01x04_Male, symbol Connector:Conn_01x04_Male
- added X3, X4: Conn_01x02_Male, symbol Connector:Conn_01x02_Male
- J2: value phase_out -> phase out
Connections:
- net +60V: now reaches Q1.2 (D), Q2.2 (D), Q3.2 (D), Q4.2 (D)
- net +60V: now also J1. (Pin_1), U1.5 (+60V); no longer J1.1 (Pin_1), U1. (phase)
- net at Q5.1 (G): now also U1.21 (Q5)
- net phase: now reaches Q1.3 (S), Q2.3 (S), Q3.3 (S), Q4.3 (S), Q5.2 (D), Q6.2 (D), Q7.2 (D), Q8.2 (D)
- net phase: now also J2. (Pin_1), U1.16 (phase); no longer J2.1 (Pin_1), U1. (phase)
- net -60V: now reaches Q5.3 (S), Q6.3 (S), Q7.3 (S), Q8.3 (S)
- net -60V: now also J3. (Pin_1), U1.20 (-60V); no longer J3.1 (Pin_1), U1. (phase)
- net G1: now reaches Q1.1 (G)
- net G1: now also U1.1 (Q1)
- net G2: now reaches Q2.1 (G)
- net G2: now also U1.2 (Q2)
- net at Q7.1 (G): now also U1.13 (Q7)
- net at Q8.1 (G): now also U1.10 (Q8)
- net G3: now reaches Q3.1 (G)
- net G3: now also U1.6 (Q3)
- net at Q6.1 (G): now also U1.17 (Q6)
- net G4: now reaches Q4.1 (G)
- net G4: now also U1.9 (Q4)
- new net: R2.2, U1.18 (t2-)
- new net: R2.1, U1.19 (t2+)
- new net: R1.1, U1.3 (t1+)
- new net: R1.2, U1.4 (t1-)
- new net +12V: U1. (fan-), X1.1 (Pin_1)
- new net +24V: U1. (fan-), X2.1 (Pin_1)
- new net -12V: U1. (fan-), X1.3 (Pin_3)
- new net -24V: U1. (fan-), X2.3 (Pin_3)
- new net fan+: U1. (fan-), X3.1 (Pin_1), X4.1 (Pin_1)
- new net fan-: U1. (fan-), X3.2 (Pin_2), X4.2 (Pin_2)
Other:
- moved on the sheet: Q1, Q2, Q3, Q4

Commit message: Signed-off-by: Dmitry Ponyatov <dponyatov@samsa.local>
Parts:
- U1: footprint (none) -> pwm_meson:pwm_meson0
- X1, X2: footprint (none) -> terminal:PLS-4
- X3, X4: footprint (none) -> terminal:CWF-2
Connections:
- net fan+: now also U1.14A (fan+), X3.2 (Pin_2), X4.2 (Pin_2); no longer U1. (fan-), X3.1 (Pin_1), X4.1 (Pin_1)
- net fan-: now also U1.14J (fan-), X3.1 (Pin_1), X4.1 (Pin_1); no longer U1. (fan-), X3.2 (Pin_2), X4.2 (Pin_2)
- net G5: now reaches Q5.1 (G), U1.21 (Q5)
- net G8: now reaches Q8.1 (G), U1.10 (Q8)
- net G7: now reaches Q7.1 (G), U1.13 (Q7)
- net G6: now reaches Q6.1 (G), U1.17 (Q6)
- net t2-: now reaches R2.2, U1.18 (t2-)
- net t2+: now reaches R2.1, U1.19 (t2+)
- net t1+: now reaches R1.1, U1.3 (t1+)
- net t1-: now reaches R1.2, U1.4 (t1-)

Commit message: Signed-off-by: Dmitry Ponyatov <dponyatov@samsa.local>
Parts:
- removed R1, R2: Thermistor, symbol Device:Thermistor
- added R1, R2: B57045K, Resistor_THT:R_Axial_DIN0411_L9.9mm_D3.6mm_P7.62mm_Vertical, symbol sensor:B57045K
Connections:
- net t1+: now also U1.7A (t1+), R1.1; no longer U1.3 (t1+)
- net t1-: now also U1.5A (t1-), R1.2; no longer U1.4 (t1-)
- net t2+: now also U1.7J (t2+), R2.1; no longer U1.19 (t2+)
- net t2-: now also U1.5J (t2-), R2.2; no longer U1.18 (t2-)
Changed lines of the file:
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@@
     (pin "16")
     (pin "17")
-    (pin "18")
-    (pin "19")
     (pin "2")
     (pin "20")
     (pin "21")
-    (pin "3")
-    (pin "4")
+    (pin "5J")
     (pin "5")
+    (pin "5A")
     (pin "6")
+    (pin "7A")
+    (pin "7J")
     (pin "9")
-  )
-  (symbol (lib_id "Device:Thermistor") (at 30.48 67.31 0) (unit 1)
-    (in_bom yes) (on_board yes) (fields_autoplaced)
-    (property "Reference" "R1" (id 0) (at 34.29 66.0399 0)
-      (effects (font (size 1.27 1.27)) (justify left))
-    )
-    (property "Value" "Thermistor" (id 1) (at 34.29 68.5799 0)
-      (effects (font (size 1.27 1.27)) (justify left))
-    )
-    (property "Footprint" "" (id 2) (at 30.48 67.31 0)
-      (effects (font (size 1.27 1.27)) hide)
-    )
-    (property "Datasheet" "~" (id 3) (at 30.48 67.31 0)
-      (effects (font (size 1.27 1.27)) hide)
-    )
-    (pin "1")
-    (pin "2")
   )
   (symbol (lib_id "mosfet:IRFB4321PBF") (at 149.86 64.77 0) (unit 1)
@@
     (pin "2")
   )
-  (symbol (lib_id "Device:Thermistor") (at 30.48 90.17 0) (unit 1)
-    (in_bom yes) (on_board yes) (fields_autoplaced)
-    (property "Reference" "R2" (id 0) (at 34.29 88.8999 0)
-      (effects (font (size 1.27 1.27)) (justify left))
-    )
-    (property "Value" "Thermistor" (id 1) (at 34.29 91.4399 0)
-      (effects (font (size 1.27 1.27)) (justify left))
-    )
-    (property "Footprint" "" (id 2) (at 30.48 90.17 0)
-      (effects (font (size 1.27 1.27)) hide)
-    )
-    (property "Datasheet" "~" (id 3) (at 30.48 90.17 0)
-      (effects (font (size 1.27 1.27)) hide)
-    )
-    (pin "1")
-    (pin "2")
-  )
   (symbol (lib_id "mosfet:IRFB4321PBF") (at 180.34 64.77 0) (unit 1)
     (in_bom yes) (on_board yes) (fields_autoplaced)
@@
     (pin "2")
     (pin "3")
+  )
+  (symbol (lib_id "sensor:B57045K") (at 30.48 90.17 0) (unit 1)
+    (in_bom yes) (on_board yes) (fields_autoplaced)
+    (property "Reference" "R2" (id 0) (at 34.29 88.8999 0)
+      (effects (font (size 1.27 1.27)) (justify left))
+    )
+    (property "Value" "B57045K" (id 1) (at 34.29 91.4399 0)
+      (effects (font (size 1.27 1.27)) (justify left))
+    )
+    (property "Footprint" "Resistor_THT:R_Axial_DIN0411_L9.9mm_D3.6mm_P7.62mm_Vertical" (id 2) (at 30.48 90.17 0)
+      (effects (font (size 1.27 1.27)) hide)
+    )
+    (property "Datasheet" "~" (id 3) (at 30.48 90.17 0)
+      (effects (font (size 1.27 1.27)) hide)
+    )
+    (pin "1")
+    (pin "2")
+  )
+  (symbol (lib_id "sensor:B57045K") (at 30.48 67.31 0) (unit 1)
+    (in_bom yes) (on_board yes) (fields_autoplaced)
+    (property "Reference" "R1" (id 0) (at 34.29 66.0399 0)
+      (effects (font (size 1.27 1.27)) (justify left))
+    )
+    (property "Value" "B57045K" (id 1) (at 34.29 68.5799 0)
+      (effects (font (size 1.27 1.27)) (justify left))
+    )
+    (property "Footprint" "Resistor_THT:R_Axial_DIN0411_L9.9mm_D3.6mm_P7.62mm_Vertical" (id 2) (at 30.48 67.31 0)
+      (effects (font (size 1.27 1.27)) hide)
+    )
+    (property "Datasheet" "~" (id 3) (at 30.48 67.31 0)
+      (effects (font (size 1.27 1.27)) hide)
+    )
+    (pin "1")
+    (pin "2")
   )
   (sheet_instances
@@
       (reference "Q8") (unit 1) (value "IRFB4321PBF") (footprint "Package_TO_SOT_THT:TO-220-3_Vertical")
     )
-    (path "/71964cfc-48ce-4fe9-94ee-9ee7dbd4487f"
-      (reference "R1") (unit 1) (value "Thermistor") (footprint "")
-    )
-    (path "/b32ed2dc-11a0-40f1-95a6-a7364d676455"
-      (reference "R2") (unit 1) (value "Thermistor") (footprint "")
+    (path "/ffb71a1d-5ce2-4a48-9050-1d23c97fdb02"
+      (reference "R1") (unit 1) (value "B57045K") (footprint "Resistor_THT:R_Axial_DIN0411_L9.9mm_D3.6mm_P7.62mm_Vertical")
+    )
+    (path "/f79b5acd-04d0-4fa1-9a9c-1af4a1811c54"
+      (reference "R2") (unit 1) (value "B57045K") (footprint "Resistor_THT:R_Axial_DIN0411_L9.9mm_D3.6mm_P7.62mm_Vertical")
     )
     (path "/67c256b8-88b9-4e93-9bf7-2bbf5ffafcf0"

Commit message: Signed-off-by: Dmitry Ponyatov <dponyatov@samsa.local>
Connections:
- net +12V: now also U1.20J (+12V); no longer U1. (-24V)
- net -12V: now also U1.22J (-12V); no longer U1. (-24V)
Changed lines of the file:
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@@
-    (pin "")
-    (pin "")
     (pin "")
     (pin "")
@@
     (pin "2")
     (pin "20")
+    (pin "20J")
     (pin "21")
-    (pin "5J")
+    (pin "22J")
     (pin "5")
     (pin "5A")
+    (pin "5J")
     (pin "6")
     (pin "7A")

Commit message: Signed-off-by: Dmitry Ponyatov <dponyatov@samsa.local>
Connections:
- net +24V: now also U1.16A (+24V); no longer U1. (-24V)
- net -24V: now also U1.16J (-24V); no longer U1. (-24V)
Changed lines of the file:
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@@
       (effects (font (size 1.27 1.27)) hide)
     )
-    (pin "")
-    (pin "")
+    (pin "16A")
+    (pin "16J")
     (pin "1")
     (pin "10")

Commit message: Signed-off-by: Dmitry Ponyatov <dponyatov@samsa.local>
Connections:
- net +60V: now also U1.10A (+60V); no longer U1.5 (+60V)
- net G1: now also U1.1A (Q1); no longer U1.1 (Q1)
- net G2: now also U1.3A (Q2); no longer U1.2 (Q2)
- net G3: now also U1.12A (Q3); no longer U1.6 (Q3)
- net G4: now also U1.20A (Q4); no longer U1.9 (Q4)
Changed lines of the file:
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@@
       (effects (font (size 1.27 1.27)) hide)
     )
-    (pin "16A")
-    (pin "16J")
-    (pin "1")
+    (pin "1A")
     (pin "10")
     (pin "13")
@@
     (pin "14J")
     (pin "16")
+    (pin "16A")
+    (pin "16J")
     (pin "17")
-    (pin "2")
+    (pin "3A")
     (pin "20")
     (pin "20J")
     (pin "21")
     (pin "22J")
-    (pin "5")
+    (pin "10A")
     (pin "5A")
     (pin "5J")
-    (pin "6")
+    (pin "12A")
     (pin "7A")
     (pin "7J")
-    (pin "9")
+    (pin "20A")
   )
   (symbol (lib_id "mosfet:IRFB4321PBF") (at 149.86 64.77 0) (unit 1)

Commit message: Signed-off-by: Dmitry Ponyatov <dponyatov@samsa.local>
Parts:
- J1, J3: footprint (none) -> terminal:screw_M4; symbol terminal:Screw_1xM4 -> terminal:Screw_M4
- J2: value phase out -> phase; footprint (none) -> terminal:screw_M4; symbol terminal:Screw_1xM4 -> terminal:Screw_M4
- Q1, Q2, Q3, Q4: footprint Package_TO_SOT_THT:TO-220-3_Vertical -> mosfet:TO-220AB
- Q5, Q6, Q7, Q8: footprint Package_TO_SOT_THT:TO-220-3_Vertical -> mosfet:TO-220AB_m
Connections:
- net +60V: now also J1.1 (Pin_1); no longer J1. (Pin_1)
- net -60V: now also J3.1 (Pin_1), U1.3J (-60V); no longer J3. (Pin_1), U1.20 (-60V)
- net G5: now also U1.1J (Q5); no longer U1.21 (Q5)
- net G6: now also U1.9J (Q6); no longer U1.17 (Q6)
- net G7: now also U1.18J (Q7); no longer U1.13 (Q7)
- net G8: now also U1.24J (Q8); no longer U1.10 (Q8)
- net phase: now also J2.1 (Pin_1), U1.12J (phase); no longer J2. (Pin_1), U1.16 (phase)
Changed lines of the file:
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@@
     (effects (font (size 1.27 1.27)) (justify left bottom))
   )
-  (symbol (lib_name "Screw_1xM4_1") (lib_id "terminal:Screw_1xM4") (at 238.76 78.74 0) (unit 1)
+  (symbol (lib_id "terminal:Screw_M4") (at 238.76 78.74 0) (unit 1)
     (in_bom yes) (on_board yes) (fields_autoplaced)
     (property "Reference" "J2" (id 0) (at 241.3 77.4699 0)
       (effects (font (size 1.27 1.27)) (justify left))
     )
-    (property "Value" "phase out" (id 1) (at 241.3 80.0099 0)
-      (effects (font (size 1.27 1.27)) (justify left))
-    )
-    (property "Footprint" "" (id 2) (at 238.76 78.74 0)
+    (property "Value" "phase" (id 1) (at 241.3 80.0099 0)
+      (effects (font (size 1.27 1.27)) (justify left))
+    )
+    (property "Footprint" "terminal:screw_M4" (id 2) (at 237.49 81.28 0)
       (effects (font (size 1.27 1.27)) hide)
     )
@@
       (effects (font (size 1.27 1.27)) hide)
     )
-    (pin "")
-  )
-  (symbol (lib_name "Screw_1xM4_1") (lib_id "terminal:Screw_1xM4") (at 238.76 57.15 0) (unit 1)
+    (pin "1")
+  )
+  (symbol (lib_id "terminal:Screw_M4") (at 238.76 57.15 0) (unit 1)
     (in_bom yes) (on_board yes) (fields_autoplaced)
     (property "Reference" "J1" (id 0) (at 241.3 55.8799 0)
@@
       (effects (font (size 1.27 1.27)) (justify left))
     )
-    (property "Footprint" "" (id 2) (at 238.76 57.15 0)
+    (property "Footprint" "terminal:screw_M4" (id 2) (at 237.49 59.69 0)
       (effects (font (size 1.27 1.27)) hide)
     )
@@
       (effects (font (size 1.27 1.27)) hide)
     )
-    (pin "")
+    (pin "1")
   )
   (symbol (lib_id "mosfet:IRFB4321PBF") (at 116.84 87.63 0) (unit 1)
@@
       (effects (font (size 1.27 1.27)) (justify left))
     )
-    (property "Footprint" "Package_TO_SOT_THT:TO-220-3_Vertical" (id 2) (at 123.19 89.535 0)
+    (property "Footprint" "mosfet:TO-220AB_m" (id 2) (at 123.19 89.535 0)
       (effects (font (size 1.27 1.27) italic) (justify left) hide)
     )
@@
       (effects (font (size 1.27 1.27)) (justify left))
     )
-    (property "Footprint" "Package_TO_SOT_THT:TO-220-3_Vertical" (id 2) (at 123.19 66.675 0)
+    (property "Footprint" "mosfet:TO-220AB" (id 2) (at 123.19 66.675 0)
       (effects (font (size 1.27 1.27) italic) (justify left) hide)
     )
@@
       (effects (font (size 1.27 1.27)) (justify left))
     )
-    (property "Footprint" "pwm_meson:pwm_meson0" (id 2) (at 76.2 78.74 0)
+    (property "Footprint" "pwm_meson:pwm_meson0" (id 2) (at 76.2 81.28 0)
       (effects (font (size 1.27 1.27)) hide)
     )
@@
       (effects (font (size 1.27 1.27)) hide)
     )
-    (pin "1A")
-    (pin "10")
-    (pin "13")
+    (pin "24J")
+    (pin "10A")
+    (pin "12A")
+    (pin "12J")
+    (pin "18J")
     (pin "14A")
     (pin "14J")
-    (pin "16")
     (pin "16A")
     (pin "16J")
-    (pin "17")
+    (pin "1A")
+    (pin "1J")
+    (pin "20A")
+    (pin "20J")
+    (pin "22J")
     (pin "3A")
-    (pin "20")
-    (pin "20J")
-    (pin "21")
-    (pin "22J")
-    (pin "10A")
+    (pin "3J")
     (pin "5A")
     (pin "5J")
-    (pin "12A")
     (pin "7A")
     (pin "7J")
-    (pin "20A")
+    (pin "9J")
   )
   (symbol (lib_id "mosfet:IRFB4321PBF") (at 149.86 64.77 0) (unit 1)
@@
       (effects (font (size 1.27 1.27)) (justify left))
     )
-    (property "Footprint" "Package_TO_SOT_THT:TO-220-3_Vertical" (id 2) (at 156.21 66.675 0)
+    (property "Footprint" "mosfet:TO-220AB" (id 2) (at 156.21 66.675 0)
       (effects (font (size 1.27 1.27) italic) (justify left) hide)
     )
@@
       (effects (font (size 1.27 1.27)) (justify left))
     )
-    (property "Footprint" "Package_TO_SOT_THT:TO-220-3_Vertical" (id 2) (at 186.69 89.535 0)
+    (property "Footprint" "mosfet:TO-220AB_m" (id 2) (at 186.69 89.535 0)
       (effects (font (size 1.27 1.27) italic) (justify left) hide)
     )
@@
       (effects (font (size 1.27 1.27)) (justify left))
     )
-    (property "Footprint" "Package_TO_SOT_THT:TO-220-3_Vertical" (id 2) (at 217.17 89.535 0)
+    (property "Footprint" "mosfet:TO-220AB_m" (id 2) (at 217.17 89.535 0)
       (effects (font (size 1.27 1.27) italic) (justify left) hide)
     )
@@
       (effects (font (size 1.27 1.27)) (justify left))
     )
-    (property "Footprint" "Package_TO_SOT_THT:TO-220-3_Vertical" (id 2) (at 186.69 66.675 0)
+    (property "Footprint" "mosfet:TO-220AB" (id 2) (at 186.69 66.675 0)
       (effects (font (size 1.27 1.27) italic) (justify left) hide)
     )
@@
     (pin "4")
   )
-  (symbol (lib_name "Screw_1xM4_1") (lib_id "terminal:Screw_1xM4") (at 238.76 101.6 0) (unit 1)
+  (symbol (lib_id "terminal:Screw_M4") (at 238.76 101.6 0) (unit 1)
     (in_bom yes) (on_board yes) (fields_autoplaced)
     (property "Reference" "J3" (id 0) (at 241.3 100.3299 0)
@@
       (effects (font (size 1.27 1.27)) (justify left))
     )
-    (property "Footprint" "" (id 2) (at 238.76 101.6 0)
+    (property "Footprint" "terminal:screw_M4" (id 2) (at 237.49 104.14 0)
       (effects (font (size 1.27 1.27)) hide)
     )
@@
       (effects (font (size 1.27 1.27)) hide)
     )
-    (pin "")
+    (pin "1")
   )
   (symbol (lib_id "mosfet:IRFB4321PBF") (at 149.86 87.63 0) (unit 1)
@@
       (effects (font (size 1.27 1.27)) (justify left))
     )
-    (property "Footprint" "Package_TO_SOT_THT:TO-220-3_Vertical" (id 2) (at 156.21 89.535 0)
+    (property "Footprint" "mosfet:TO-220AB_m" (id 2) (at 156.21 89.535 0)
       (effects (font (size 1.27 1.27) italic) (justify left) hide)
     )
@@
       (effects (font (size 1.27 1.27)) (justify left))
     )
-    (property "Footprint" "Package_TO_SOT_THT:TO-220-3_Vertical" (id 2) (at 217.17 66.675 0)
+    (property "Footprint" "mosfet:TO-220AB" (id 2) (at 217.17 66.675 0)
       (effects (font (size 1.27 1.27) italic) (justify left) hide)
     )
@@
   (symbol_instances
     (path "/22667c69-544a-4658-9de0-227e9f7a59ff"
-      (reference "J1") (unit 1) (value "+60V") (footprint "")
+      (reference "J1") (unit 1) (value "+60V") (footprint "terminal:screw_M4")
     )
     (path "/208563d9-099e-4500-b0ab-0fe95158f39a"
-      (reference "J2") (unit 1) (value "phase out") (footprint "")
+      (reference "J2") (unit 1) (value "phase") (footprint "terminal:screw_M4")
     )
     (path "/e5d33526-ec58-4fc5-a4b0-4886c00b27d6"
-      (reference "J3") (unit 1) (value "-60V") (footprint "")
+      (reference "J3") (unit 1) (value "-60V") (footprint "terminal:screw_M4")
     )
     (path "/4548bfaa-3e38-41d2-b802-c8a1d015231c"
-      (reference "Q1") (unit 1) (value "IRFB4321PBF") (footprint "Package_TO_SOT_THT:TO-220-3_Vertical")
+      (reference "Q1") (unit 1) (value "IRFB4321PBF") (footprint "mosfet:TO-220AB")
     )
     (path "/805dc104-45c8-4f28-85c6-a29bf180dd37"
-      (reference "Q2") (unit 1) (value "IRFB4321PBF") (footprint "Package_TO_SOT_THT:TO-220-3_Vertical")
+      (reference "Q2") (unit 1) (value "IRFB4321PBF") (footprint "mosfet:TO-220AB")
     )
     (path "/ca65c19a-1f5c-42db-a938-5f601f55048c"
-      (reference "Q3") (unit 1) (value "IRFB4321PBF") (footprint "Package_TO_SOT_THT:TO-220-3_Vertical")
+      (reference "Q3") (unit 1) (value "IRFB4321PBF") (footprint "mosfet:TO-220AB")
     )
     (path "/f54ef2e4-8aba-4967-ae1d-979b8149fb57"
-      (reference "Q4") (unit 1) (value "IRFB4321PBF") (footprint "Package_TO_SOT_THT:TO-220-3_Vertical")
+      (reference "Q4") (unit 1) (value "IRFB4321PBF") (footprint "mosfet:TO-220AB")
     )
     (path "/27d3a7a0-d6b7-487d-b0c0-9ba220769453"
-      (reference "Q5") (unit 1) (value "IRFB4321PBF") (footprint "Package_TO_SOT_THT:TO-220-3_Vertical")
+      (reference "Q5") (unit 1) (value "IRFB4321PBF") (footprint "mosfet:TO-220AB_m")
     )
     (path "/e6a227ca-6e7c-49a4-b26b-1f9ea24b3957"
-      (reference "Q6") (unit 1) (value "IRFB4321PBF") (footprint "Package_TO_SOT_THT:TO-220-3_Vertical")
+      (reference "Q6") (unit 1) (value "IRFB4321PBF") (footprint "mosfet:TO-220AB_m")
     )
     (path "/82850c45-f7db-4984-8811-e31b743e1ce8"
-      (reference "Q7") (unit 1) (value "IRFB4321PBF") (footprint "Package_TO_SOT_THT:TO-220-3_Vertical")
+      (reference "Q7") (unit 1) (value "IRFB4321PBF") (footprint "mosfet:TO-220AB_m")
     )
     (path "/9ecfa4a9-bdf3-4903-b08c-e6d2be19e0d9"
-      (reference "Q8") (unit 1) (value "IRFB4321PBF") (footprint "Package_TO_SOT_THT:TO-220-3_Vertical")
+      (reference "Q8") (unit 1) (value "IRFB4321PBF") (footprint "mosfet:TO-220AB_m")
     )
     (path "/ffb71a1d-5ce2-4a48-9050-1d23c97fdb02"
