File: pcb/pwm/pwm.kicad_sch (KiCad schematic)
At the start: 18 parts, among them J1 +60V, J2 phase, J3 -60V, Q1 IRFB4321PBF, Q2 IRFB4321PBF, Q3 IRFB4321PBF, Q4 IRFB4321PBF, Q5 IRFB4321PBF, Q6 IRFB4321PBF, Q7 IRFB4321PBF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

Commit message: Signed-off-by: Dmitry Ponyatov <dponyatov@samsa.local>
Connections:
- net +12V: now also U1.22J (+12V), X1.3 (Pin_3); no longer U1.20J (+12V), X1.1 (Pin_1)
- net +24V: now also U1.16J (+24V), X2.4 (Pin_4); no longer U1.16A (+24V), X2.1 (Pin_1)
- net -12V: now also U1.20J (-12V), X1.1 (Pin_1); no longer U1.22J (-12V), X1.3 (Pin_3)
- net -24V: now also U1.16A (-24V), X2.2 (Pin_2); no longer U1.16J (-24V), X2.3 (Pin_3)
Changed lines of the file:
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@@
     (stroke (width 0) (type default) (color 0 0 0 0))
   )
-  (wire (pts (xy 67.31 109.22) (xy 67.31 135.89))
+  (wire (pts (xy 67.31 109.22) (xy 67.31 138.43))
     (stroke (width 0) (type default) (color 0 0 0 0))
   )
@@
     (stroke (width 0) (type default) (color 0 0 0 0))
   )
-  (wire (pts (xy 64.77 109.22) (xy 64.77 140.97))
+  (wire (pts (xy 64.77 109.22) (xy 64.77 143.51))
     (stroke (width 0) (type default) (color 0 0 0 0))
   )
@@
     (stroke (width 0) (type default) (color 0 0 0 0))
   )
-  (wire (pts (xy 184.15 140.97) (xy 64.77 140.97))
+  (wire (pts (xy 184.15 143.51) (xy 64.77 143.51))
     (stroke (width 0) (type default) (color 0 0 0 0))
   )
@@
     (stroke (width 0) (type default) (color 0 0 0 0))
   )
-  (wire (pts (xy 184.15 135.89) (xy 67.31 135.89))
+  (wire (pts (xy 184.15 138.43) (xy 67.31 138.43))
     (stroke (width 0) (type default) (color 0 0 0 0))
   )
@@
     (stroke (width 0) (type default) (color 0 0 0 0))
   )
-  (label "-24V" (at 177.8 140.97 0)
-    (effects (font (size 1.27 1.27)) (justify left bottom))
-  )
-  (label "-24V" (at 64.77 110.49 270)
-    (effects (font (size 1.27 1.27)) (justify right bottom))
+  (label "+24V" (at 177.8 143.51 0)
+    (effects (font (size 1.27 1.27)) (justify left bottom))
   )
   (label "G3" (at 86.36 73.66 0)
     (effects (font (size 1.27 1.27)) (justify left bottom))
-  )
-  (label "-12V" (at 69.85 110.49 270)
-    (effects (font (size 1.27 1.27)) (justify right bottom))
-  )
-  (label "+24V" (at 67.31 110.49 270)
-    (effects (font (size 1.27 1.27)) (justify right bottom))
   )
   (label "fan-" (at 54.61 130.81 180)
@@
     (effects (font (size 1.27 1.27)) (justify left bottom))
   )
-  (label "+12V" (at 177.8 116.84 0)
-    (effects (font (size 1.27 1.27)) (justify left bottom))
-  )
-  (label "+12V" (at 72.39 110.49 270)
-    (effects (font (size 1.27 1.27)) (justify right bottom))
+  (label "-12V" (at 177.8 116.84 0)
+    (effects (font (size 1.27 1.27)) (justify left bottom))
   )
   (label "fan+" (at 54.61 133.35 180)
@@
     (effects (font (size 1.27 1.27)) (justify left bottom))
   )
-  (label "-12V" (at 177.8 121.92 0)
+  (label "+12V" (at 177.8 121.92 0)
     (effects (font (size 1.27 1.27)) (justify left bottom))
   )
@@
     (effects (font (size 1.27 1.27)) (justify left bottom))
   )
-  (label "+24V" (at 177.8 135.89 0)
+  (label "-24V" (at 177.8 138.43 0)
     (effects (font (size 1.27 1.27)) (justify left bottom))
   )
@@
     (effects (font (size 1.27 1.27)) (justify left bottom))
   )
-  (symbol (lib_id "terminal:Screw_M4") (at 238.76 78.74 0) (unit 1)
+  (symbol (lib_name "Screw_M4_2") (lib_id "terminal:Screw_M4") (at 238.76 78.74 0) (unit 1)
     (in_bom yes) (on_board yes) (fields_autoplaced)
     (property "Reference" "J2" (id 0) (at 241.3 77.4699 0)
@@
     (pin "1")
   )
-  (symbol (lib_id "terminal:Screw_M4") (at 238.76 57.15 0) (unit 1)
+  (symbol (lib_name "Screw_M4_1") (lib_id "terminal:Screw_M4") (at 238.76 57.15 0) (unit 1)
     (in_bom yes) (on_board yes) (fields_autoplaced)
     (property "Reference" "J1" (id 0) (at 241.3 55.8799 0)
@@
       (effects (font (size 1.27 1.27)) hide)
     )
-    (pin "24J")
     (pin "10A")
     (pin "12A")
     (pin "12J")
-    (pin "18J")
     (pin "14A")
     (pin "14J")
     (pin "16A")
     (pin "16J")
+    (pin "18J")
     (pin "1A")
     (pin "1J")
@@
     (pin "20J")
     (pin "22J")
+    (pin "24J")
     (pin "3A")
     (pin "3J")
