File: pcb/proto/proto.kicad_pcb (KiCad board)
At the start: 2 copper layers, 50.8 x 25.4 mm, 1 part, among them J1 USB_B_Mini

Commit message: Signed-off-by: Dmitry Ponyatov <ponyatov@example.com>
Parts:
- removed J1: USB_B_Mini, Connector_USB:USB_Mini-B_DS1104
- added C1: 10uF, Capacitor_SMD:C_1206_3216Metric_Pad1.33x1.80mm_HandSolder, F.Cu at (110.5, 81.3)
- added C2: 10uF, Capacitor_SMD:C_1206_3216Metric_Pad1.33x1.80mm_HandSolder, F.Cu at (118.2, 79.0)
- added C3: 0805, Capacitor_SMD:C_0805_2012Metric_Pad1.18x1.45mm_HandSolder, F.Cu at (122.4, 98.1)
- added C4: 0603, Capacitor_SMD:C_0603_1608Metric_Pad1.08x0.95mm_HandSolder, F.Cu at (113.0, 99.6)
- added C5: C_Polarized_Small, Capacitor_SMD:C_0402_1005Metric_Pad0.74x0.62mm_HandSolder, F.Cu at (132.3, 87.8)
- added C6: C_Polarized_Small, Capacitor_SMD:C_0402_1005Metric_Pad0.74x0.62mm_HandSolder, F.Cu at (123.4, 86.9)
- added JP1: slave, Resistor_SMD:R_0201_0603Metric, F.Cu at (112.8, 90.1)
- added U1: AMS1117-3.3, Package_TO_SOT_SMD:SOT-223-3_TabPin2, F.Cu at (118.2, 83.5)
- added U2: CH340C, Package_SO:SOIC-16_3.9x9.9mm_P1.27mm, F.Cu at (117.3, 94.9)
- added U3: F030F4Px, Package_SO:TSSOP-20_4.4x6.5mm_P0.65mm, F.Cu at (128.0, 87.8)
- added USB1: USB_B_Mini, Connector_USB:USB_Mini-B_DS1104, F.Cu at (107.9, 88.9)
- added XTAL1: HC-49S, crystal:Crystal_HC49-2P_mill, B.Cu at (129.8, 80.3)
Routing:
- net /GND: track 0.00 -> 124.1 mm, vias 0 -> 4
- net (no net): track 0.00 -> 51.6 mm
- net /VCC3: track 0.00 -> 48.4 mm
- net /D+: track 0.00 -> 13.2 mm
- net /D-: track 0.00 -> 13.2 mm
- net /VCC5: track 0.00 -> 10.4 mm
- net /X-: track 0.00 -> 8.71 mm
- net /X+: track 0.00 -> 8.01 mm
- net /ID: track 0.00 -> 2.32 mm

Commit message: Signed-off-by: Dmitry Ponyatov <ponyatov@example.com>
Parts:
- JP1: footprint Resistor_SMD:R_0201_0603Metric -> Resistor_SMD:R_0402_1005Metric_Pad0.72x0.64mm_HandSolder
- moved JP1 0.15 mm to (112.8, 90.3)
Routing:
- net /GND: track 124.1 -> 130.4 mm
- net /X+: track 8.01 -> 9.07 mm
- net /X-: track 8.71 -> 9.37 mm

Commit message: Signed-off-by: Dmitry Ponyatov <ponyatov@example.com>
Parts:
- moved C4 0.10 mm to (112.9, 99.6)
Changed lines of the file:
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@@
   )
   (footprint "Capacitor_SMD:C_0603_1608Metric_Pad1.08x0.95mm_HandSolder" (layer "F.Cu")
-    (at 112.9792 99.568 -90)
+    (at 112.8776 99.568 -90)
     (descr "Capacitor SMD 0603 (1608 Metric), square (rectangular) end terminal, IPC_7351 nominal with elongated pad for handsoldering. (Body size source: IPC-SM-782 page 76, https://www.pcb-3d.com/wordpress/wp-content/uploads/ipc-sm-782a_amendment_1_and_2.pdf), generated with kicad-footprint-generator")
     (tags "capacitor handsolder")
@@
   (segment (start 108.0052 93.9604) (end 109.9252 93.9604) (width 0.5) (layer "F.Cu") (net 31))
   (segment (start 124.4854 77.3938) (end 122.2502 77.3938) (width 0.5) (layer "F.Cu") (net 31))
+  (segment (start 119.7864 100.1268) (end 119.1768 100.7364) (width 0.5) (layer "F.Cu") (net 31))
   (segment (start 102.9252 93.9604) (end 104.4252 93.9604) (width 0.5) (layer "F.Cu") (net 31))
   (segment (start 104.4252 93.9604) (end 105.1052 93.2804) (width 0.5) (layer "F.Cu") (net 31))
@@
   (segment (start 133.4472 87.6496) (end 132.736 88.3608) (width 0.5) (layer "F.Cu") (net 31))
   (segment (start 104.4252 83.8004) (end 105.1052 84.4804) (width 0.5) (layer "F.Cu") (net 31))
-  (segment (start 119.7864 100.1268) (end 119.1768 100.7364) (width 0.5) (layer "F.Cu") (net 31))
-  (segment (start 119.1768 100.7364) (end 113.2851 100.7364) (width 0.5) (layer "F.Cu") (net 31))
   (segment (start 131.884717 88.3499) (end 131.693017 88.1582) (width 0.3) (layer "F.Cu") (net 31))
   (segment (start 114.3552 79.3554) (end 114.9902 79.9904) (width 0.5) (layer "F.Cu") (net 31))
@@
   (segment (start 118.1579 77.4192) (end 116.6027 78.9744) (width 0.5) (layer "F.Cu") (net 31))
   (segment (start 108.9302 81.2604) (end 108.9302 80.0814) (width 0.5) (layer "F.Cu") (net 31))
+  (segment (start 113.1835 100.7364) (end 112.8776 100.4305) (width 0.5) (layer "F.Cu") (net 31))
   (segment (start 106.5784 86.3092) (end 107.8992 84.9884) (width 0.5) (layer "F.Cu") (net 31))
   (segment (start 133.4472 85.0856) (end 133.4472 87.6496) (width 0.5) (layer "F.Cu") (net 31))
@@
   (segment (start 108.0052 93.9604) (end 105.7852 93.9604) (width 0.5) (layer "F.Cu") (net 31))
   (segment (start 120.396 100.7364) (end 119.7864 100.1268) (width 0.5) (layer "F.Cu") (net 31))
-  (segment (start 113.2851 100.7364) (end 112.9792 100.4305) (width 0.5) (layer "F.Cu") (net 31))
   (segment (start 105.7852 83.8004) (end 105.1052 84.4804) (width 0.5) (layer "F.Cu") (net 31))
   (segment (start 111.7852 90.5) (end 110.4992 90.5) (width 0.3) (layer "F.Cu") (net 31))
@@
   (segment (start 111.104 96.3988) (end 111.104 99.4468) (width 0.2) (layer "F.Cu") (net 31))
   (segment (start 104.9992 93.3) (end 104.9992 84.5) (width 0.5) (layer "F.Cu") (net 31))
+  (segment (start 119.1768 100.7364) (end 113.1835 100.7364) (width 0.5) (layer "F.Cu") (net 31))
   (segment (start 123.3932 84.3788) (end 123.3932 86.3513) (width 0.5) (layer "F.Cu") (net 31))
   (segment (start 124.7648 82.7024) (end 122.1232 80.0608) (width 0.5) (layer "F.Cu") (net 31))

Commit message: Signed-off-by: Dmitry Ponyatov <ponyatov@example.com>
Parts:
- added D1: 1N4148WT, Diode_SMD:D_SOD-523, F.Cu at (112.7, 96.1)
- added D2: 1N4148WT, Diode_SMD:D_SOD-523, F.Cu at (110.8, 96.1)
- C3: value 0805 -> 0603; footprint Capacitor_SMD:C_0805_2012Metric_Pad1.18x1.45mm_HandSolder -> Capacitor_SMD:C_0603_1608Metric_Pad1.08x0.95mm_HandSolder
- C4: value 0603 -> 0805; footprint Capacitor_SMD:C_0603_1608Metric_Pad1.08x0.95mm_HandSolder -> Capacitor_SMD:C_0805_2012Metric_Pad1.18x1.45mm_HandSolder
- JP1: footprint Resistor_SMD:R_0402_1005Metric_Pad0.72x0.64mm_HandSolder -> Resistor_SMD:R_0201_0603Metric
- moved C4 0.25 mm to (112.6, 99.6)
- moved JP1 0.10 mm to (112.8, 90.4)
Connections:
- C1 pad 1: /VCC5 -> /VUSB
- C4 pad 1: /VCC3 -> /VCC5
- U1 pad 3: /VCC5 -> /VUSB
- U2 pad 16: /VCC3 -> /VCC5
- USB1 pad 1: /VCC5 -> /VUSB
Routing:
- net /VUSB: track 0.00 -> 19.5 mm, vias 0 -> 2
- net /VCC3: track 48.4 -> 38.3 mm
- net /VCC5: track 10.4 -> 7.29 mm, vias 0 -> 1
- net Net-(D1-Pad1): track 0.00 -> 2.46 mm
