File: pcb/proto/proto.kicad_sch (KiCad schematic)
At the start: 1 part

Commit message: Signed-off-by: Dmitry Ponyatov <ponyatov@example.com>
Parts:
- added C1, C2: 10uF, Capacitor_SMD:C_1206_3216Metric_Pad1.33x1.80mm_HandSolder, symbol Device:C_Polarized
- added C3: 0805, Capacitor_SMD:C_0805_2012Metric_Pad1.18x1.45mm_HandSolder, symbol Device:C_Polarized_Small
- added C4: 0603, Capacitor_SMD:C_0603_1608Metric_Pad1.08x0.95mm_HandSolder, symbol Device:C_Polarized_Small
- added C5, C6: C_Polarized_Small, Capacitor_SMD:C_0402_1005Metric_Pad0.74x0.62mm_HandSolder, symbol Device:C_Polarized_Small
- added JP1: slave, Resistor_SMD:R_0201_0603Metric, symbol Jumper:SolderJumper_2_Open
- added U1: AMS1117-3.3, Package_TO_SOT_SMD:SOT-223-3_TabPin2, symbol Regulator_Linear:AMS1117-3.3
- added U2: CH340C, Package_SO:SOIC-16_3.9x9.9mm_P1.27mm, symbol Interface_USB:CH340C
- added U3: STM32F030F4Px, Package_SO:TSSOP-20_4.4x6.5mm_P0.65mm, symbol MCU_ST_STM32F0:STM32F030F4Px
- added XTAL1: HC-49S, crystal:Crystal_HC49-2P_mill, symbol crystal:HC-49S
- USB1: renamed from J?; footprint Connector_USB:USB3_Micro-B_Connfly_DS1104-01 -> Connector_USB:USB_Mini-B_DS1104
Connections:
- net VCC5: now reaches USB1.1 (VBUS)
- net VCC5: now also C1.1, U1.3 (VI)
- net D-: now reaches USB1.2 (D-)
- net D-: now also U2.6 (UD-)
- net D+: now reaches USB1.3 (D+)
- net D+: now also U2.5 (UD+)
- net ID: now reaches USB1.4 (ID)
- net ID: now also JP1.2 (B)
- net GND: now reaches USB1.5 (GND)
- net GND: now also USB1.6 (Shield), C1.2, C2.2, C3.2, C4.2, C5.2, C6.2, JP1.1 (A), U1.1 (GND), U2.1 (GND), U3.15 (VSS), XTAL1.3
- new net VCC3: C2.1, C3.1, C4.1, C5.1, C6.1, U1.2 (VO), U2.16 (VCC), U2.4 (V3), U3.16 (VDD), U3.5 (VDDA)
- new net X+: U3.2 (PF0), XTAL1.2
- new net X-: U3.3 (PF1), XTAL1.1

Commit message: Signed-off-by: Dmitry Ponyatov <ponyatov@example.com>
Parts:
- U3: value STM32F030F4Px -> F030F4Px
Changed lines of the file:
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@@
       (effects (font (size 1.27 1.27)) (justify left))
     )
-    (property "Value" "STM32F030F4Px" (id 1) (at 154.4194 88.9 0)
+    (property "Value" "F030F4Px" (id 1) (at 154.4194 88.9 0)
       (effects (font (size 1.27 1.27)) (justify left))
     )
@@
     )
     (path "/9c228180-21bc-4b39-b26f-0b1a0dfeee4c"
-      (reference "U3") (unit 1) (value "STM32F030F4Px") (footprint "Package_SO:TSSOP-20_4.4x6.5mm_P0.65mm")
+      (reference "U3") (unit 1) (value "F030F4Px") (footprint "Package_SO:TSSOP-20_4.4x6.5mm_P0.65mm")
     )
     (path "/2c803c1b-17e8-4d10-bf2e-c46c5b6727f7"

Commit message: Signed-off-by: Dmitry Ponyatov <ponyatov@example.com>
Parts:
- added D1, D2: 1N4148WT, Diode_SMD:D_SOD-523, symbol Diode:1N4148WT
- renumbered C4 to C3, C3 to C4
Connections:
- net VCC3: no longer C4.1, U2.16 (VCC)
- net VCC5: now also C4.1, U2.16 (VCC), D2.1 (K); no longer C1.1, U1.3 (VI), USB1.1 (VBUS)
- new net: D1.1 (K), D2.2 (A)
- new net VUSB: C1.1, D1.2 (A), U1.3 (VI), USB1.1 (VBUS)
Changed lines of the file:
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@@
   (junction (at 104.14 95.25) (diameter 0) (color 0 0 0 0)
   )
+  (junction (at 104.14 50.8) (diameter 0) (color 0 0 0 0)
+  )
   (junction (at 101.6 53.34) (diameter 0) (color 0 0 0 0)
   )
@@
   (junction (at 101.6 46.99) (diameter 0) (color 0 0 0 0)
   )
-  (junction (at 104.14 50.8) (diameter 0) (color 0 0 0 0)
+  (junction (at 63.5 46.99) (diameter 0) (color 0 0 0 0)
   )
   (junction (at 152.4 43.18) (diameter 0) (color 0 0 0 0)
@@
   (junction (at 72.39 58.42) (diameter 0) (color 0 0 0 0)
   )
-  (junction (at 104.14 46.99) (diameter 0) (color 0 0 0 0)
-  )
   (wire (pts (xy 55.88 81.28) (xy 55.88 95.25))
     (stroke (width 0) (type default) (color 0 0 0 0))
@@
     (stroke (width 0) (type default) (color 0 0 0 0))
   )
+  (wire (pts (xy 104.14 36.83) (xy 104.14 50.8))
+    (stroke (width 0) (type default) (color 0 0 0 0))
+  )
   (wire (pts (xy 152.4 43.18) (xy 154.94 43.18))
     (stroke (width 0) (type default) (color 0 0 0 0))
@@
     (stroke (width 0) (type default) (color 0 0 0 0))
   )
+  (wire (pts (xy 82.55 36.83) (xy 63.5 36.83))
+    (stroke (width 0) (type default) (color 0 0 0 0))
+  )
   (wire (pts (xy 139.7 78.74) (xy 135.89 78.74))
     (stroke (width 0) (type default) (color 0 0 0 0))
@@
     (stroke (width 0) (type default) (color 0 0 0 0))
   )
-  (wire (pts (xy 101.6 46.99) (xy 104.14 46.99))
-    (stroke (width 0) (type default) (color 0 0 0 0))
-  )
   (wire (pts (xy 63.5 72.39) (xy 66.04 72.39))
     (stroke (width 0) (type default) (color 0 0 0 0))
@@
     (stroke (width 0) (type default) (color 0 0 0 0))
   )
+  (wire (pts (xy 90.17 36.83) (xy 93.98 36.83))
+    (stroke (width 0) (type default) (color 0 0 0 0))
+  )
   (wire (pts (xy 63.5 58.42) (xy 63.5 46.99))
     (stroke (width 0) (type default) (color 0 0 0 0))
@@
     (stroke (width 0) (type default) (color 0 0 0 0))
   )
+  (wire (pts (xy 63.5 36.83) (xy 63.5 46.99))
+    (stroke (width 0) (type default) (color 0 0 0 0))
+  )
   (wire (pts (xy 55.88 81.28) (xy 58.42 81.28))
     (stroke (width 0) (type default) (color 0 0 0 0))
@@
     (stroke (width 0) (type default) (color 0 0 0 0))
   )
-  (wire (pts (xy 104.14 46.99) (xy 104.14 50.8))
-    (stroke (width 0) (type default) (color 0 0 0 0))
-  )
   (wire (pts (xy 173.99 38.1) (xy 173.99 95.25))
     (stroke (width 0) (type default) (color 0 0 0 0))
@@
     (stroke (width 0) (type default) (color 0 0 0 0))
   )
-  (wire (pts (xy 104.14 46.99) (xy 152.4 46.99))
+  (wire (pts (xy 101.6 36.83) (xy 104.14 36.83))
+    (stroke (width 0) (type default) (color 0 0 0 0))
+  )
+  (wire (pts (xy 101.6 46.99) (xy 152.4 46.99))
     (stroke (width 0) (type default) (color 0 0 0 0))
   )
@@
     (effects (font (size 1.27 1.27)) (justify left bottom))
   )
+  (label "VCC5" (at 104.14 41.91 0)
+    (effects (font (size 1.27 1.27)) (justify left bottom))
+  )
   (label "ID" (at 66.04 76.2 0)
     (effects (font (size 1.27 1.27)) (justify left bottom))
@@
     (effects (font (size 1.27 1.27)) (justify left bottom))
   )
-  (label "VCC5" (at 63.5 49.53 180)
+  (label "VUSB" (at 63.5 49.53 180)
     (effects (font (size 1.27 1.27)) (justify right bottom))
   )
@@
   (symbol (lib_id "Device:C_Polarized_Small") (at 109.22 50.8 90) (unit 1)
     (in_bom yes) (on_board yes)
-    (property "Reference" "C3" (id 0) (at 106.68 49.53 90))
+    (property "Reference" "C4" (id 0) (at 106.68 49.53 90))
     (property "Value" "0805" (id 1) (at 108.6739 46.99 90))
     (property "Footprint" "Capacitor_SMD:C_0805_2012Metric_Pad1.18x1.45mm_HandSolder" (id 2) (at 109.22 50.8 0)
@@
   (symbol (lib_id "Device:C_Polarized_Small") (at 111.76 53.34 90) (unit 1)
     (in_bom yes) (on_board yes)
-    (property "Reference" "C4" (id 0) (at 114.3 54.61 90))
+    (property "Reference" "C3" (id 0) (at 114.3 54.61 90))
     (property "Value" "0603" (id 1) (at 111.2139 49.53 90)
       (effects (font (size 1.27 1.27)) hide)
@@
     (pin "9")
   )
+  (symbol (lib_id "Diode:1N4148WT") (at 86.36 36.83 180) (unit 1)
+    (in_bom yes) (on_board yes) (fields_autoplaced)
+    (property "Reference" "D1" (id 0) (at 86.36 30.48 0))
+    (property "Value" "1N4148WT" (id 1) (at 86.36 33.02 0))
+    (property "Footprint" "Diode_SMD:D_SOD-523" (id 2) (at 86.36 32.385 0)
+      (effects (font (size 1.27 1.27)) hide)
+    )
+    (property "Datasheet" "https://www.diodes.com/assets/Datasheets/ds30396.pdf" (id 3) (at 86.36 36.83 0)
+      (effects (font (size 1.27 1.27)) hide)
+    )
+    (pin "1")
+    (pin "2")
+  )
   (symbol (lib_id "Device:C_Polarized_Small") (at 157.48 38.1 90) (unit 1)
     (in_bom yes) (on_board yes)
@@
     )
     (property "Datasheet" "~" (id 3) (at 157.48 38.1 0)
+      (effects (font (size 1.27 1.27)) hide)
+    )
+    (pin "1")
+    (pin "2")
+  )
+  (symbol (lib_id "Diode:1N4148WT") (at 97.79 36.83 180) (unit 1)
+    (in_bom yes) (on_board yes) (fields_autoplaced)
+    (property "Reference" "D2" (id 0) (at 97.79 30.48 0))
+    (property "Value" "1N4148WT" (id 1) (at 97.79 33.02 0))
+    (property "Footprint" "Diode_SMD:D_SOD-523" (id 2) (at 97.79 32.385 0)
+      (effects (font (size 1.27 1.27)) hide)
+    )
+    (property "Datasheet" "https://www.diodes.com/assets/Datasheets/ds30396.pdf" (id 3) (at 97.79 36.83 0)
       (effects (font (size 1.27 1.27)) hide)
     )
@@
       (reference "C2") (unit 1) (value "10uF") (footprint "Capacitor_SMD:C_1206_3216Metric_Pad1.33x1.80mm_HandSolder")
     )
+    (path "/32201266-c8d7-4d68-abab-ed38d0b5536e"
+      (reference "C3") (unit 1) (value "0603") (footprint "Capacitor_SMD:C_0603_1608Metric_Pad1.08x0.95mm_HandSolder")
+    )
     (path "/30d3dacd-4777-4fcb-ba43-580b979785c7"
-      (reference "C3") (unit 1) (value "0805") (footprint "Capacitor_SMD:C_0805_2012Metric_Pad1.18x1.45mm_HandSolder")
-    )
-    (path "/32201266-c8d7-4d68-abab-ed38d0b5536e"
-      (reference "C4") (unit 1) (value "0603") (footprint "Capacitor_SMD:C_0603_1608Metric_Pad1.08x0.95mm_HandSolder")
+      (reference "C4") (unit 1) (value "0805") (footprint "Capacitor_SMD:C_0805_2012Metric_Pad1.18x1.45mm_HandSolder")
     )
     (path "/c132144a-dea4-4cfc-b78f-82f08cb596a9"
@@
       (reference "C6") (unit 1) (value "C_Polarized_Small") (footprint "Capacitor_SMD:C_0402_1005Metric_Pad0.74x0.62mm_HandSolder")
     )
+    (path "/bacd8f51-3da5-4511-99fa-5e589b6d5b21"
+      (reference "D1") (unit 1) (value "1N4148WT") (footprint "Diode_SMD:D_SOD-523")
+    )
+    (path "/c8521663-3c85-4ef4-a3d7-7d58b3169fc7"
+      (reference "D2") (unit 1) (value "1N4148WT") (footprint "Diode_SMD:D_SOD-523")
+    )
     (path "/6546db3e-3346-4386-905b-9c0edfb02d8d"
