File: pcb/bat/bat.kicad_pcb (KiCad board)
At the start: 2 copper layers, 50.8 x 25.4 mm, 14 parts, among them U1 AMS1117-3.3, U2 CH340C, U3 F030F4Px

Commit message: Signed-off-by: Dmitry Ponyatov <ponyatov@example.com>
Parts:
- added R1: 0R, Resistor_SMD:R_0201_0603Metric, F.Cu at (123.4, 87.1)
- added U4: AP9101CK, Package_TO_SOT_SMD:SOT-23-5, F.Cu at (144.8, 88.9)
- XTAL1: value HC-49S -> 8Mhz
- moved C6 1.58 mm to (123.4, 85.3)
Connections:
- U3 pad 10: unconnected-(U3-Pad10) -> /LED
- U3 pad 5: /VCC3 -> /VDDA
- U3 pad 6: unconnected-(U3-Pad6) -> /A0
- U3 pad 7: unconnected-(U3-Pad7) -> /A1
- U3 pad 8: unconnected-(U3-Pad8) -> /A2
- U3 pad 9: unconnected-(U3-Pad9) -> /A3
Routing:
- net /VCC3: track 38.3 -> 32.0 mm
- net /VDDA: track 0.00 -> 1.67 mm
- net /GND: track 130.5 -> 128.9 mm

Commit message: Signed-off-by: Dmitry Ponyatov <ponyatov@example.com>
Connections:
- C1 pad 2: /GND -> GND
- C2 pad 2: /GND -> GND
- C3 pad 2: /GND -> GND
- C4 pad 2: /GND -> GND
- C5 pad 2: /GND -> GND
- C6 pad 2: /GND -> GND
- JP1 pad 1: /GND -> GND
- U1 pad 1: /GND -> GND
- U2 pad 1: /GND -> GND
- U3 pad 15: /GND -> GND
- U4 pad 3: unconnected-(U4-Pad3) -> GND
- USB1 pad 5: /GND -> GND
- USB1 pad 6: /GND -> GND
Routing:
- net /GND: track 128.9 -> 0.00 mm, vias 4 -> 0
- net GND: track 0.00 -> 122.8 mm, vias 0 -> 4
- net (no net): track 51.6 -> 57.7 mm

Commit message: Signed-off-by: Dmitry Ponyatov <ponyatov@example.com>
Parts:
- added Q1: FS8205A, Package_SO:TSSOP-8_4.4x3mm_P0.65mm, F.Cu at (141.7, 95.0)
- U4: value AP9101CK -> AP9101CK-AHTRG1
Changed lines of the file:
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@@
   (net 40 "unconnected-(U4-Pad5)")
   (net 41 "GND")
+  (net 42 "unconnected-(Q1-Pad1)")
+  (net 43 "Net-(Q1-Pad2)")
+  (net 44 "unconnected-(Q1-Pad3)")
+  (net 45 "unconnected-(Q1-Pad4)")
+  (net 46 "unconnected-(Q1-Pad6)")
   (footprint "Package_SO:SOIC-16_3.9x9.9mm_P1.27mm" (layer "F.Cu")
     (at 117.3016 94.9256 180)
@@
     )
   )
+  (footprint "Package_SO:TSSOP-8_4.4x3mm_P0.65mm" (layer "F.Cu")
+    (at 141.732 95.004)
+    (descr "TSSOP, 8 Pin (JEDEC MO-153 Var AA https://www.jedec.org/document_search?search_api_views_fulltext=MO-153), generated with kicad-footprint-generator ipc_gullwing_generator.py")
+    (tags "TSSOP SO")
+    (property "Availability" "In Stock")
+    (property "Check_prices" "https://www.snapeda.com/parts/FS8205/Fortune+Semiconductor/view-part/?ref=eda")
+    (property "ChipDip" "https://www.chipdip.ru/product0/8035566278")
+    (property "Description" "\nDual N-Channel Enhancement Mode Power MOSFET\n")
+    (property "MANUFACTURER" "Fortune")
+    (property "MAXIMUM_PACKAGE_HEIGHT" "1.45mm")
+    (property "MF" "Fortune Semiconductor")
+    (property "MP" "FS8205")
+    (property "PARTREV" "1.9")
+    (property "Package" "Package")
+    (property "Price" "None")
+    (property "STANDARD" "IPC-7351B")
+    (property "Sheetfile" "bat.kicad_sch")
+    (property "Sheetname" "")
+    (property "SnapEDA_Link" "https://www.snapeda.com/parts/FS8205/Fortune+Semiconductor/view-part/?ref=snap")
+    (attr smd)
+    (fp_text reference "Q1" (at 0 -2.45) (layer "F.SilkS")
+      (effects (font (size 1 1) (thickness 0.15)))
+    )
+    (fp_text value "FS8205A" (at 0 2.45) (layer "F.Fab")
+      (effects (font (size 1 1) (thickness 0.15)))
+    )
+    (fp_text user "${REFERENCE}" (at 0 0) (layer "F.Fab")
+      (effects (font (size 1 1) (thickness 0.15)))
+    )
+    (fp_line (start 0 1.61) (end 2.2 1.61) (layer "F.SilkS") (width 0.12))
+    (fp_line (start 0 1.61) (end -2.2 1.61) (layer "F.SilkS") (width 0.12))
+    (fp_line (start 0 -1.61) (end -3.6 -1.61) (layer "F.SilkS") (width 0.12))
+    (fp_line (start 0 -1.61) (end 2.2 -1.61) (layer "F.SilkS") (width 0.12))
+    (fp_line (start 3.85 -1.75) (end -3.85 -1.75) (layer "F.CrtYd") (width 0.05))
+    (fp_line (start -3.85 -1.75) (end -3.85 1.75) (layer "F.CrtYd") (width 0.05))
+    (fp_line (start -3.85 1.75) (end 3.85 1.75) (layer "F.CrtYd") (width 0.05))
+    (fp_line (start 3.85 1.75) (end 3.85 -1.75) (layer "F.CrtYd") (width 0.05))
+    (fp_line (start -2.2 1.5) (end -2.2 -0.75) (layer "F.Fab") (width 0.1))
+    (fp_line (start -1.45 -1.5) (end 2.2 -1.5) (layer "F.Fab") (width 0.1))
+    (fp_line (start -2.2 -0.75) (end -1.45 -1.5) (layer "F.Fab") (width 0.1))
+    (fp_line (start 2.2 1.5) (end -2.2 1.5) (layer "F.Fab") (width 0.1))
+    (fp_line (start 2.2 -1.5) (end 2.2 1.5) (layer "F.Fab") (width 0.1))
+    (pad "1" smd roundrect (at -2.8625 -0.975) (size 1.475 0.4) (layers "F.Cu" "F.Paste" "F.Mask") (roundrect_rratio 0.25)
+      (net 42 "unconnected-(Q1-Pad1)") (pintype "passive"))
+    (pad "2" smd roundrect (at -2.8625 -0.325) (size 1.475 0.4) (layers "F.Cu" "F.Paste" "F.Mask") (roundrect_rratio 0.25)
+      (net 43 "Net-(Q1-Pad2)") (pintype "passive"))
+    (pad "3" smd roundrect (at -2.8625 0.325) (size 1.475 0.4) (layers "F.Cu" "F.Paste" "F.Mask") (roundrect_rratio 0.25)
+      (net 44 "unconnected-(Q1-Pad3)") (pintype "passive"))
+    (pad "4" smd roundrect (at -2.8625 0.975) (size 1.475 0.4) (layers "F.Cu" "F.Paste" "F.Mask") (roundrect_rratio 0.25)
+      (net 45 "unconnected-(Q1-Pad4)") (pintype "passive"))
+    (pad "5" smd roundrect (at 2.8625 0.975) (size 1.475 0.4) (layers "F.Cu" "F.Paste" "F.Mask") (roundrect_rratio 0.25)
+      (net 43 "Net-(Q1-Pad2)") (pintype "passive"))
+    (pad "6" smd roundrect (at 2.8625 0.325) (size 1.475 0.4) (layers "F.Cu" "F.Paste" "F.Mask") (roundrect_rratio 0.25)
+      (net 46 "unconnected-(Q1-Pad6)") (pintype "passive"))
+    (pad "7" smd roundrect (at 2.8625 -0.325) (size 1.475 0.4) (layers "F.Cu" "F.Paste" "F.Mask") (roundrect_rratio 0.25))
+    (pad "8" smd roundrect (at 2.8625 -0.975) (size 1.475 0.4) (layers "F.Cu" "F.Paste" "F.Mask") (roundrect_rratio 0.25))
+    (model "${KICAD6_3DMODEL_DIR}/Package_SO.3dshapes/TSSOP-8_4.4x3mm_P0.65mm.wrl"
+      (offset (xyz 0 0 0))
+      (scale (xyz 1 1 1))
+      (rotate (xyz 0 0 0))
+    )
+  )
   (footprint "Package_TO_SOT_SMD:SOT-223-3_TabPin2" (layer "F.Cu")
     (at 118.1652 83.5464)
@@
       (effects (font (size 1 1) (thickness 0.15)))
     )
-    (fp_text value "AP9101CK" (at 0 2.4) (layer "F.SilkS")
-      (effects (font (size 1 1) (thickness 0.15)))
-    )
+    (fp_text value "AP9101CK-AHTRG1" (at 0 2.4) (layer "F.SilkS") hide
+      (effects (font (size 1 1) (thickness 0.15)))
+    )

Commit message: Signed-off-by: Dmitry Ponyatov <ponyatov@example.com>
Parts:
- added BT1: LP232635, Connector_PinHeader_2.54mm:PinHeader_1x02_P2.54mm_Horizontal, B.Cu at (141.6, 97.2)
- added F1: JK-nSMD, Resistor_SMD:R_1206_3216Metric, F.Cu at (146.7, 97.2)
- added U5: TP4056, power:SOP127P600X175-9N, F.Cu at (133.6, 97.8)
- moved Q1 14.1 mm to (140.0, 81.0)
Connections:
- Q1 pad 1: unconnected-(Q1-Pad1) -> Net-(Q1-Pad1)
- Q1 pad 3: unconnected-(Q1-Pad3) -> Net-(Q1-Pad2)
- Q1 pad 5: Net-(Q1-Pad2) -> unconnected-(Q1-Pad5)
- Q1 pad 6: unconnected-(Q1-Pad6) -> Net-(Q1-Pad6)
- Q1 pad 7: (no net) -> Net-(Q1-Pad6)
- Q1 pad 8: (no net) -> Net-(Q1-Pad1)
Routing:
- net /BAT-: track 0.00 -> 3.62 mm

Commit message: Signed-off-by: Dmitry Ponyatov <dponyatov@gmail.com>
Parts:
- added C10: 10pF, Resistor_SMD:R_0402_1005Metric_Pad0.72x0.64mm_HandSolder, F.Cu at (123.7, 97.7)
- added C11: 10pF, Resistor_SMD:R_0402_1005Metric_Pad0.72x0.64mm_HandSolder, F.Cu at (111.0, 99.6)
- added C12: 10pF, Resistor_SMD:R_0402_1005Metric_Pad0.72x0.64mm_HandSolder, F.Cu at (129.5, 83.8)
- added C13: 10pF, Resistor_SMD:R_0402_1005Metric_Pad0.72x0.64mm_HandSolder, F.Cu at (126.7, 83.8)
- added C7: 10pF, Resistor_SMD:R_0402_1005Metric_Pad0.72x0.64mm_HandSolder, F.Cu at (111.3, 80.2)
- added C8: 10pF, Resistor_SMD:R_0402_1005Metric_Pad0.72x0.64mm_HandSolder, F.Cu at (119.1, 79.2)
- added C9: 100nF, Resistor_SMD:R_0805_2012Metric_Pad1.20x1.40mm_HandSolder, F.Cu at (141.0, 91.4)
- added J1: SWD, Connector_PinHeader_2.54mm:PinHeader_1x04_P2.54mm_Horizontal, F.Cu at (134.6, 82.6)
- added R2: 2.7K, Resistor_SMD:R_0402_1005Metric_Pad0.72x0.64mm_HandSolder, F.Cu at (136.1, 88.4)
- added R3: 330, Resistor_SMD:R_0805_2012Metric_Pad1.20x1.40mm_HandSolder, F.Cu at (137.4, 92.7)
- C6: value C_Polarized_Small -> 10pF; footprint Capacitor_SMD:C_0402_1005Metric_Pad0.74x0.62mm_HandSolder -> Resistor_SMD:R_0402_1005Metric_Pad0.72x0.64mm_HandSolder
- moved D2 13.2 mm to (124.0, 94.5), turned to 0 degrees
- moved D1 11.0 mm to (120.1, 87.9), turned to 180 degrees
- moved Q1 9.06 mm to (146.7, 87.1), turned to 90 degrees
- moved C2 3.10 mm to (115.1, 79.0)
- moved U4 2.52 mm to (143.0, 87.1)
- moved F1 2.51 mm to (144.5, 95.9), turned to 90 degrees
- moved C1 0.53 mm to (110.5, 81.8)
- moved JP1 0.34 mm to (112.9, 90.1)
Connections:
- net /BAT- renamed Net-(BT1-Pad1)
- net Net-(Q1-Pad1) renamed /D12
- C1 pad 1: /VUSB -> /VCC5
- C2 pad 1: /VCC3 -> /VCC3U
- D1 pad 1: Net-(D1-Pad1) -> /VCC3
- D1 pad 2: /VUSB -> /VCC3U
- D2 pad 1: /VCC5 -> /VCC3
- D2 pad 2: Net-(D1-Pad1) -> /BAT+
- F1 pad 2: unconnected-(F1-Pad2) -> /S1
- Q1 pad 2: Net-(Q1-Pad2) -> /S1
- Q1 pad 3: Net-(Q1-Pad2) -> /S1
- Q1 pad 4: unconnected-(Q1-Pad4) -> /G+
- Q1 pad 5: unconnected-(Q1-Pad5) -> /G-
- Q1 pad 6: Net-(Q1-Pad6) -> GND
- Q1 pad 7: Net-(Q1-Pad6) -> GND
- U1 pad 2: /VCC3 -> /VCC3U
- U1 pad 3: /VUSB -> /VCC5
- U2 pad 2: unconnected-(U2-Pad2) -> /TxD
- U2 pad 3: unconnected-(U2-Pad3) -> /RxD
- U3 pad 19: unconnected-(U3-Pad19) -> /SWDIO
- U3 pad 20: unconnected-(U3-Pad20) -> /SWCLK
- U3 pad 8: /A2 -> /TxD
- U3 pad 9: /A3 -> /RxD
- U4 pad 1: unconnected-(U4-Pad1) -> /VM
- U4 pad 2: unconnected-(U4-Pad2) -> /VDCK
- U4 pad 3: GND -> /S1
- U4 pad 4: unconnected-(U4-Pad4) -> /G+
- U4 pad 5: unconnected-(U4-Pad5) -> /G-
- USB1 pad 1: /VUSB -> /VCC5
Routing:
- net GND: track 122.8 -> 177.2 mm, vias 4 -> 6
- net /VCC5: track 7.29 -> 30.5 mm, vias 1 -> 2
- net /VCC3U: track 0.00 -> 20.2 mm, vias 0 -> 1
- net /VUSB: track 19.5 -> 0.00 mm, vias 2 -> 0
- net /BAT+: track 0.00 -> 18.0 mm, vias 0 -> 2
- net /S1: track 0.00 -> 15.8 mm
- net /VCC3: track 32.0 -> 46.8 mm, vias 0 -> 1
- net /SWDIO: track 0.00 -> 10.1 mm
- net /VDCK: track 0.00 -> 9.90 mm
- net /SWCLK: track 0.00 -> 7.85 mm
- net /D12: track 0.00 -> 7.84 mm, vias 0 -> 2
- net /VM: track 0.00 -> 6.23 mm
- net /G-: track 0.00 -> 5.99 mm
- net /G+: track 0.00 -> 5.88 mm
- net Net-(D1-Pad1): track 2.46 -> 0.00 mm
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
Commit message: Signed-off-by: Dmitry Ponyatov <dponyatov@gmail.com>
Parts:
- added C14: 10pF, Resistor_SMD:R_0402_1005Metric_Pad0.72x0.64mm_HandSolder, F.Cu at (127.3, 93.2)
- added JP2: reset, Resistor_SMD:R_0201_0603Metric, F.Cu at (127.0, 91.9)
- moved C3 3.94 mm to (123.4, 94.3)
- moved C10 3.13 mm to (124.7, 94.7)
- moved D2 2.81 mm to (126.7, 94.2)
- moved R2 1.48 mm to (134.9, 89.2)
- moved C5 0.97 mm to (133.0, 88.4)
Connections:
- U3 pad 11: unconnected-(U3-Pad11) -> /SCK
- U3 pad 12: unconnected-(U3-Pad12) -> /MISO
- U3 pad 13: unconnected-(U3-Pad13) -> /MOSI
- U3 pad 17: unconnected-(U3-Pad17) -> /SCL
- U3 pad 18: unconnected-(U3-Pad18) -> /SDA
- U3 pad 4: unconnected-(U3-Pad4) -> /RST
Routing:
- net GND: track 177.2 -> 192.9 mm
- net /TxD: track 0.00 -> 14.9 mm, vias 0 -> 2
- net /RST: track 0.00 -> 13.9 mm, vias 0 -> 2
- net /RxD: track 0.00 -> 11.7 mm, vias 0 -> 2
- net /SDA: track 0.00 -> 6.14 mm, vias 0 -> 1
- net /SCL: track 0.00 -> 4.92 mm, vias 0 -> 1
- net /BAT+: track 18.0 -> 15.1 mm
- net /VCC3: track 46.8 -> 45.3 mm
- net /VM: track 6.23 -> 7.57 mm
Other:
- board text added: "3.3v"
- board text added: "CLK"
- board text added: "DIO"
- board text added: "GND"
