File: pcb/bat/bat.kicad_pcb (KiCad board)
At the start: 2 copper layers, 50.8 x 25.4 mm, 32 parts, among them J1 SWD, Q1 FS8205A, U1 AMS1117-3.3, U2 CH340C, U3 F030F4Px, U4 AP9101CK-AHTRG1, U5 TP4056

Commit message: Signed-off-by: Dmitry Ponyatov <ponyatov@example.com>
Parts:
- moved JP1 0.10 mm to (112.9, 90.2)
Routing:
- net (no net): track 57.7 -> 54.9 mm
