File: pcb/bat/bat.kicad_sch (KiCad schematic)
At the start: 14 parts, among them U1 AMS1117-3.3, U2 CH340C, U3 F030F4Px

Commit message: Signed-off-by: Dmitry Ponyatov <ponyatov@example.com>
Parts:
- added C7: 10pF, symbol Device:C_Small
- added J1: SWD, symbol Connector:Conn_01x04_Male
- added R1: 0R, Resistor_SMD:R_0201_0603Metric, symbol Device:R_Small
- added U4: AP9101CK-AHTRG1, Package_TO_SOT_SMD:SOT-23-5, symbol Battery_Management:AP9101CK-AHTRG1
- XTAL1: value HC-49S -> 8Mhz; Part (none) -> HC-49S
Connections:
- net GND: now also J1.1 (Pin_1)
- net VCC3: now also J1.4 (Pin_4), R1.1; no longer U3.5 (VDDA)
- net LED: now reaches U3.10 (PA4)
- net A0: now reaches U3.6 (PA0)
- net A1: now reaches U3.7 (PA1)
- net A2: now reaches U3.8 (PA2)
- net A3: now reaches U3.9 (PA3)
- new net SWCLK: J1.2 (Pin_2)
- new net SWDIO: J1.3 (Pin_3)
- new net VDDA: R1.2, U3.5 (VDDA)

Commit message: Signed-off-by: Dmitry Ponyatov <ponyatov@example.com>
Parts:
- added BT1: Battery_Cell, symbol Device:Battery_Cell
- added Q1: FS8205A, FS8205:SOT95P280X145-6N, symbol Fortune_Semiconductor:FS8205A
Connections:
- net GND: now also U4.3 (VSS)
- new net: Q1.2, Q1.5
Changed lines of the file:
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@@
   (junction (at 114.3 50.8) (diameter 0) (color 0 0 0 0)
   )
+  (junction (at 55.88 95.25) (diameter 0) (color 0 0 0 0)
+  )
   (junction (at 81.28 46.99) (diameter 0) (color 0 0 0 0)
   )
@@
     (stroke (width 0) (type default) (color 0 0 0 0))
   )
+  (wire (pts (xy 87.63 143.51) (xy 87.63 151.13))
+    (stroke (width 0) (type default) (color 0 0 0 0))
+  )
   (wire (pts (xy 104.14 36.83) (xy 104.14 50.8))
     (stroke (width 0) (type default) (color 0 0 0 0))
@@
   )
   (wire (pts (xy 81.28 46.99) (xy 101.6 46.99))
+    (stroke (width 0) (type default) (color 0 0 0 0))
+  )
+  (wire (pts (xy 55.88 95.25) (xy 55.88 97.79))
     (stroke (width 0) (type default) (color 0 0 0 0))
   )
@@
   (label "A2" (at 177.8 58.42 0)
     (effects (font (size 1.27 1.27)) (justify left bottom))
+  )
+  (symbol (lib_id "Device:Battery_Cell") (at 36.83 140.97 0) (unit 1)
+    (in_bom yes) (on_board yes) (fields_autoplaced)
+    (property "Reference" "BT1" (id 0) (at 40.64 137.6679 0)
+      (effects (font (size 1.27 1.27)) (justify left))
+    )
+    (property "Value" "Battery_Cell" (id 1) (at 40.64 140.2079 0)
+      (effects (font (size 1.27 1.27)) (justify left))
+    )
+    (property "Footprint" "" (id 2) (at 36.83 139.446 90)
+      (effects (font (size 1.27 1.27)) hide)
+    )
+    (property "Datasheet" "~" (id 3) (at 36.83 139.446 90)
+      (effects (font (size 1.27 1.27)) hide)
+    )
+    (pin "1")
+    (pin "2")
   )
   (symbol (lib_id "Connector:USB_B_Mini") (at 55.88 67.31 0) (unit 1)
@@
     (pin "1")
     (pin "2")
+  )
+  (symbol (lib_id "power:GND") (at 87.63 151.13 0) (unit 1)
+    (in_bom yes) (on_board yes) (fields_autoplaced)
+    (property "Reference" "#PWR0102" (id 0) (at 87.63 157.48 0)
+      (effects (font (size 1.27 1.27)) hide)
+    )
+    (property "Value" "GND" (id 1) (at 87.63 156.21 0))
+    (property "Footprint" "" (id 2) (at 87.63 151.13 0)
+      (effects (font (size 1.27 1.27)) hide)
+    )
+    (property "Datasheet" "" (id 3) (at 87.63 151.13 0)
+      (effects (font (size 1.27 1.27)) hide)
+    )
+    (pin "1")
   )
   (symbol (lib_id "Device:C_Polarized") (at 77.47 58.42 270) (unit 1)
@@
     (pin "9")
   )
+  (symbol (lib_id "power:GND") (at 55.88 97.79 0) (unit 1)
+    (in_bom yes) (on_board yes) (fields_autoplaced)
+    (property "Reference" "#PWR0101" (id 0) (at 55.88 104.14 0)
+      (effects (font (size 1.27 1.27)) hide)
+    )
+    (property "Value" "GND" (id 1) (at 55.88 102.87 0))
+    (property "Footprint" "" (id 2) (at 55.88 97.79 0)
+      (effects (font (size 1.27 1.27)) hide)
+    )
+    (property "Datasheet" "" (id 3) (at 55.88 97.79 0)
+      (effects (font (size 1.27 1.27)) hide)
+    )
+    (pin "1")
+  )
   (symbol (lib_id "Diode:1N4148WT") (at 86.36 36.83 180) (unit 1)
     (in_bom yes) (on_board yes) (fields_autoplaced)
@@
     (pin "5")
   )
+  (symbol (lib_id "Fortune_Semiconductor:FS8205A") (at 87.63 167.64 270) (unit 1)
+    (in_bom yes) (on_board yes) (fields_autoplaced)
+    (property "Reference" "Q1" (id 0) (at 83.82 167.64 90))
+    (property "Value" "FS8205A" (id 1) (at 81.28 167.64 90))
+    (property "Footprint" "FS8205:SOT95P280X145-6N" (id 2) (at 87.63 167.64 0)
+      (effects (font (size 1.27 1.27)) (justify bottom) hide)
+    )
+    (property "Datasheet" "https://static.chipdip.ru/lib/333/DOC050333523.pdf" (id 3) (at 87.63 167.64 0)
+      (effects (font (size 1.27 1.27)) hide)
+    )
+    (property "MF" "Fortune Semiconductor" (id 4) (at 87.63 167.64 0)
+      (effects (font (size 1.27 1.27)) (justify bottom) hide)
+    )
+    (property "MAXIMUM_PACKAGE_HEIGHT" "1.45mm" (id 5) (at 87.63 167.64 0)
+      (effects (font (size 1.27 1.27)) (justify bottom) hide)
+    )
+    (property "Package" "Package" (id 6) (at 87.63 167.64 0)
+      (effects (font (size 1.27 1.27)) (justify bottom) hide)
+    )
+    (property "Price" "None" (id 7) (at 87.63 167.64 0)
+      (effects (font (size 1.27 1.27)) (justify bottom) hide)
+    )
+    (property "Check_prices" "https://www.snapeda.com/parts/FS8205/Fortune+Semiconductor/view-part/?ref=eda" (id 8) (at 87.63 167.64 0)
+      (effects (font (size 1.27 1.27)) (justify bottom) hide)
+    )
+    (property "STANDARD" "IPC-7351B" (id 9) (at 87.63 167.64 0)
+      (effects (font (size 1.27 1.27)) (justify bottom) hide)
+    )
+    (property "PARTREV" "1.9" (id 10) (at 87.63 167.64 0)
+      (effects (font (size 1.27 1.27)) (justify bottom) hide)
+    )
+    (property "SnapEDA_Link" "https://www.snapeda.com/parts/FS8205/Fortune+Semiconductor/view-part/?ref=snap" (id 11) (at 87.63 167.64 0)
+      (effects (font (size 1.27 1.27)) (justify bottom) hide)
+    )
+    (property "MP" "FS8205" (id 12) (at 87.63 167.64 0)
+      (effects (font (size 1.27 1.27)) (justify bottom) hide)
+    )
+    (property "Description" "\nDual N-Channel Enhancement Mode Power MOSFET\n" (id 13) (at 87.63 167.64 0)
+      (effects (font (size 1.27 1.27)) (justify bottom) hide)
+    )
+    (property "Availability" "In Stock" (id 14) (at 87.63 167.64 0)
+      (effects (font (size 1.27 1.27)) (justify bottom) hide)
+    )
+    (property "MANUFACTURER" "Fortune" (id 15) (at 87.63 167.64 0)
+      (effects (font (size 1.27 1.27)) (justify bottom) hide)
+    )
+    (property "ChipDip" "https://www.chipdip.ru/product0/8035566278" (id 16) (at 87.63 167.64 0)
+      (effects (font (size 1.27 1.27)) hide)
+    )
+    (pin "1")
+    (pin "2")
+    (pin "3")
+    (pin "4")
+    (pin "5")
+    (pin "6")
+  )
   (sheet_instances
     (path "/" (page "1"))
   )
   (symbol_instances
+    (path "/ac668852-f7de-42f7-b974-c8be7eaf365a"
+      (reference "#PWR0101") (unit 1) (value "GND") (footprint "")
+    )
+    (path "/49421894-9ea3-427c-b0ca-573218bb6de7"
+      (reference "#PWR0102") (unit 1) (value "GND") (footprint "")
+    )
+    (path "/0f817ffa-4177-431b-aac1-ff14eb67e5ca"
+      (reference "BT1") (unit 1) (value "Battery_Cell") (footprint "")
+    )
     (path "/d8ae61c9-2753-4c85-860f-93abbe6def2d"
       (reference "C1") (unit 1) (value "10uF") (footprint "Capacitor_SMD:C_1206_3216Metric_Pad1.33x1.80mm_HandSolder")
@@
       (reference "JP1") (unit 1) (value "slave") (footprint "Resistor_SMD:R_0201_0603Metric")
     )
+    (path "/f1458993-7851-4345-9830-d97d21fc5c50"
+      (reference "Q1") (unit 1) (value "FS8205A") (footprint "FS8205:SOT95P280X145-6N")
+    )
     (path "/9bd6a370-09f4-420e-ba5c-59e81a214b65"

Commit message: Signed-off-by: Dmitry Ponyatov <ponyatov@example.com>
Parts:
- removed BT1: Battery_Cell, symbol Device:Battery_Cell
- added BT1: LP232635, Connector_PinHeader_2.54mm:PinHeader_1x02_P2.54mm_Horizontal, symbol power:LP232635
- added F1: JK-nSMD, Resistor_SMD:R_1206_3216Metric, symbol fuse:JK-nSMD
- added U5: TP4056, power:SOP127P600X175-9N, symbol power:TP4056
- Q1: footprint FS8205:SOT95P280X145-6N -> Package_SO:TSSOP-8_4.4x3mm_P0.65mm
Connections:
- net at Q1.1: now also Q1.8
- net at Q1.2: now also Q1.3; no longer Q1.5
- net at Q1.6: now also Q1.7
- new net BAT+: BT1.2 (+)
- new net BAT-: BT1.1 (-), F1.1

Commit message: Signed-off-by: Dmitry Ponyatov <dponyatov@gmail.com>
Parts:
- removed C6: C_Polarized_Small, Capacitor_SMD:C_0402_1005Metric_Pad0.74x0.62mm_HandSolder, symbol Device:C_Polarized_Small
- added C10, C11, C12, C13, C6, C8: 10pF, Resistor_SMD:R_0402_1005Metric_Pad0.72x0.64mm_HandSolder, symbol Device:C_Small
- added C9: 100nF, Resistor_SMD:R_0805_2012Metric_Pad1.20x1.40mm_HandSolder, symbol Device:C_Small
- added R2: 2.7K, Resistor_SMD:R_0402_1005Metric_Pad0.72x0.64mm_HandSolder, symbol Device:R
- added R3: 330, Resistor_SMD:R_0805_2012Metric_Pad1.20x1.40mm_HandSolder, symbol Device:R_Small
- C7: footprint (none) -> Resistor_SMD:R_0402_1005Metric_Pad0.72x0.64mm_HandSolder
- J1: footprint (none) -> Connector_PinHeader_2.54mm:PinHeader_1x04_P2.54mm_Horizontal
Connections:
- net A2 is gone; now on net TxD: U3.8 (PA2)
- net A3 is gone; now on net RxD: U3.9 (PA3)
- net BAT+: now also D2.2 (A), R3.1
- net BAT-: now also F1.2, Q1.2, Q1.3, U4.3 (VSS), C9.1; no longer BT1.1 (-), F1.1
- net GND: now also C7.2, Q1.6, Q1.7, C10.1, C11.2, C12.1, C13.1, C6.2, C8.1, R2.2; no longer U4.3 (VSS)
- net SWCLK: now also U3.20 (PA14)
- net SWDIO: now also U3.19 (PA13)
- net VCC3: now also D1.1 (K), D2.1 (K), C10.2, C6.1; no longer C2.1, U1.2 (VO)
- net VCC5: now also C1.1, C7.1, U1.3 (VI), USB1.1 (VBUS), C11.1; no longer D2.1 (K)
- net X+: now also C13.2
- net X-: now also C12.2
- net TxD: now reaches U2.2 (TXD)
- net RxD: now reaches U2.3 (RXD)
- net VM: now reaches U4.1 (VM)
- net VM: now also R2.1
- net VDCK: now reaches U4.2 (VDD)
- net VDCK: now also C9.2, R3.2
- net G+: now reaches U4.4 (DO)
- net G+: now also Q1.4
- net G-: now reaches U4.5 (CO)
- net G-: now also Q1.5
- net D12: now reaches Q1.1, Q1.8
- removed net VUSB: C1.1, D1.2 (A), U1.3 (VI), USB1.1 (VBUS)
- new net: BT1.1 (-), F1.1
- new net VCC3U: C2.1, C8.2, D1.2 (A), U1.2 (VO)
Other:
- moved on the sheet: BT1, C3, C7, D1, D2, F1, Q1, U5

Commit message: Signed-off-by: Dmitry Ponyatov <dponyatov@gmail.com>
Connections:
- net SCK: now reaches U3.11 (PA5)
- net MISO: now reaches U3.12 (PA6)
- net MOSI: now reaches U3.13 (PA7)
- net SCL: now reaches U3.17 (PA9)
- net SDA: now reaches U3.18 (PA10)
Changed lines of the file:
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@@
   (junction (at 101.6 46.99) (diameter 0) (color 0 0 0 0)
   )
+  (bus_entry (at 182.88 66.04) (size 2.54 2.54)
+    (stroke (width 0) (type default) (color 0 0 0 0))
+  )
+  (bus_entry (at 182.88 76.2) (size 2.54 2.54)
+    (stroke (width 0) (type default) (color 0 0 0 0))
+  )
   (bus_entry (at 185.42 36.83) (size 2.54 2.54)
     (stroke (width 0) (type default) (color 0 0 0 0))
@@
     (stroke (width 0) (type default) (color 0 0 0 0))
   )
+  (bus_entry (at 182.88 73.66) (size 2.54 2.54)
+    (stroke (width 0) (type default) (color 0 0 0 0))
+  )
   (bus_entry (at 182.88 58.42) (size 2.54 2.54)
     (stroke (width 0) (type default) (color 0 0 0 0))
   )
+  (bus_entry (at 182.88 68.58) (size 2.54 2.54)
+    (stroke (width 0) (type default) (color 0 0 0 0))
+  )
+  (bus_entry (at 182.88 71.12) (size 2.54 2.54)
+    (stroke (width 0) (type default) (color 0 0 0 0))
+  )
   (bus_entry (at 182.88 78.74) (size 2.54 2.54)
     (stroke (width 0) (type default) (color 0 0 0 0))
@@
     (stroke (width 0) (type default) (color 0 0 0 0))
   )
+  (wire (pts (xy 165.1 76.2) (xy 182.88 76.2))
+    (stroke (width 0) (type default) (color 0 0 0 0))
+  )
   (wire (pts (xy 97.79 133.35) (xy 104.14 133.35))
     (stroke (width 0) (type default) (color 0 0 0 0))
@@
     (stroke (width 0) (type default) (color 0 0 0 0))
   )
+  (bus (pts (xy 185.42 71.12) (xy 185.42 73.66))
+    (stroke (width 0) (type default) (color 0 0 0 0))
+  )
   (bus (pts (xy 185.42 63.5) (xy 185.42 66.04))
     (stroke (width 0) (type default) (color 0 0 0 0))
@@
     (stroke (width 0) (type default) (color 0 0 0 0))
   )
+  (wire (pts (xy 165.1 68.58) (xy 182.88 68.58))
+    (stroke (width 0) (type default) (color 0 0 0 0))
+  )
   (wire (pts (xy 129.54 71.12) (xy 135.89 71.12))
     (stroke (width 0) (type default) (color 0 0 0 0))
@@
     (stroke (width 0) (type default) (color 0 0 0 0))
   )
+  (wire (pts (xy 165.1 71.12) (xy 182.88 71.12))
+    (stroke (width 0) (type default) (color 0 0 0 0))
+  )
   (wire (pts (xy 152.4 86.36) (xy 152.4 95.25))
     (stroke (width 0) (type default) (color 0 0 0 0))
@@
     (stroke (width 0) (type default) (color 0 0 0 0))
   )
+  (bus (pts (xy 185.42 76.2) (xy 185.42 78.74))
+    (stroke (width 0) (type default) (color 0 0 0 0))
+  )
   (wire (pts (xy 139.7 76.2) (xy 139.7 78.74))
     (stroke (width 0) (type default) (color 0 0 0 0))
@@
     (stroke (width 0) (type default) (color 0 0 0 0))
   )
+  (bus (pts (xy 185.42 78.74) (xy 185.42 81.28))
+    (stroke (width 0) (type default) (color 0 0 0 0))
+  )
   (wire (pts (xy 135.89 71.12) (xy 139.7 71.12))
     (stroke (width 0) (type default) (color 0 0 0 0))
@@
     (stroke (width 0) (type default) (color 0 0 0 0))
   )
+  (bus (pts (xy 185.42 68.58) (xy 185.42 71.12))
+    (stroke (width 0) (type default) (color 0 0 0 0))
+  )
   (wire (pts (xy 135.89 78.74) (xy 135.89 77.47))
     (stroke (width 0) (type default) (color 0 0 0 0))
@@
     (stroke (width 0) (type default) (color 0 0 0 0))
   )
+  (wire (pts (xy 165.1 73.66) (xy 182.88 73.66))
+    (stroke (width 0) (type default) (color 0 0 0 0))
+  )
   (wire (pts (xy 45.72 140.97) (xy 45.72 143.51))
     (stroke (width 0) (type default) (color 0 0 0 0))
@@
     (stroke (width 0) (type default) (color 0 0 0 0))
   )
+  (bus (pts (xy 185.42 73.66) (xy 185.42 76.2))
+    (stroke (width 0) (type default) (color 0 0 0 0))
+  )
   (wire (pts (xy 52.07 127) (xy 45.72 127))
     (stroke (width 0) (type default) (color 0 0 0 0))
@@
     (stroke (width 0) (type default) (color 0 0 0 0))
   )
-  (bus (pts (xy 185.42 66.04) (xy 185.42 81.28))
+  (bus (pts (xy 185.42 66.04) (xy 185.42 68.58))
     (stroke (width 0) (type default) (color 0 0 0 0))
   )
@@
     (stroke (width 0) (type default) (color 0 0 0 0))
   )
+  (wire (pts (xy 165.1 66.04) (xy 182.88 66.04))
+    (stroke (width 0) (type default) (color 0 0 0 0))
+  )
   (wire (pts (xy 123.19 74.93) (xy 123.19 78.74))
     (stroke (width 0) (type default) (color 0 0 0 0))
@@
     (effects (font (size 1.27 1.27)) (justify left bottom))
   )
+  (label "SDA" (at 175.26 76.2 0)
+    (effects (font (size 1.27 1.27)) (justify left bottom))
+  )
   (label "A0" (at 177.8 53.34 0)
     (effects (font (size 1.27 1.27)) (justify left bottom))
@@
     (effects (font (size 1.27 1.27)) (justify left bottom))
   )
+  (label "MISO" (at 175.26 68.58 0)
+    (effects (font (size 1.27 1.27)) (justify left bottom))
+  )
   (label "ID" (at 66.04 76.2 0)
     (effects (font (size 1.27 1.27)) (justify left bottom))
@@
     (effects (font (size 1.27 1.27)) (justify left bottom))
   )
+  (label "SCL" (at 175.26 73.66 0)
+    (effects (font (size 1.27 1.27)) (justify left bottom))
+  )
   (label "TxD" (at 176.53 58.42 0)
     (effects (font (size 1.27 1.27)) (justify left bottom))
@@
   )
   (label "D12" (at 119.38 135.89 0)
+    (effects (font (size 1.27 1.27)) (justify left bottom))
+  )
+  (label "SCK" (at 175.26 66.04 0)
     (effects (font (size 1.27 1.27)) (justify left bottom))
   )
@@
     (effects (font (size 1.27 1.27)) (justify left bottom))
   )
+  (label "MOSI" (at 175.26 71.12 0)
+    (effects (font (size 1.27 1.27)) (justify left bottom))
+  )

Commit message: Signed-off-by: Dmitry Ponyatov <dponyatov@gmail.com>
Parts:
- C3: value 0603 -> 10uF
- C4: value 0805 -> 10uF
Other:
- moved on the sheet: C3
Changed lines of the file:
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@@
     (stroke (width 0) (type default) (color 0 0 0 0))
   )
-  (wire (pts (xy 90.17 53.34) (xy 88.9 53.34))
+  (wire (pts (xy 91.44 53.34) (xy 88.9 53.34))
     (stroke (width 0) (type default) (color 0 0 0 0))
   )
@@
     (stroke (width 0) (type default) (color 0 0 0 0))
   )
-  (wire (pts (xy 101.6 53.34) (xy 95.25 53.34))
+  (wire (pts (xy 101.6 53.34) (xy 96.52 53.34))
     (stroke (width 0) (type default) (color 0 0 0 0))
   )
@@
     (effects (font (size 1.27 1.27)) (justify left bottom))
   )
-  (label "VCC3U" (at 81.28 50.8 0)
+  (label "VCC3U" (at 81.28 45.72 0)
     (effects (font (size 1.27 1.27)) (justify left bottom))
   )
@@
   (symbol (lib_id "Device:C_Small") (at 114.3 53.34 90) (unit 1)
     (in_bom yes) (on_board yes)
-    (property "Reference" "C11" (id 0) (at 111.76 52.07 90))
-    (property "Value" "10pF" (id 1) (at 107.95 52.07 90))
-    (property "Footprint" "Resistor_SMD:R_0402_1005Metric_Pad0.72x0.64mm_HandSolder" (id 2) (at 114.3 53.34 0)
+    (property "Reference" "C11" (id 0) (at 116.84 52.07 90))
+    (property "Value" "10pF" (id 1) (at 118.11 54.61 90))
+    (property "Footprint" "Resistor_SMD:R_0402_1005Metric_Pad0.72x0.64mm_HandSolder" (id 2) (at 116.84 53.34 0)
       (effects (font (size 1.27 1.27)) hide)
     )
@@
     (in_bom yes) (on_board yes)
     (property "Reference" "C4" (id 0) (at 106.68 49.53 90))
-    (property "Value" "0805" (id 1) (at 108.6739 46.99 90))
+    (property "Value" "10uF" (id 1) (at 113.03 49.53 90))
     (property "Footprint" "Capacitor_SMD:C_0805_2012Metric_Pad1.18x1.45mm_HandSolder" (id 2) (at 109.22 50.8 0)
       (effects (font (size 1.27 1.27)) hide)
@@
     (pin "2")
   )
-  (symbol (lib_id "Device:C_Polarized_Small") (at 92.71 53.34 270) (unit 1)
-    (in_bom yes) (on_board yes)
-    (property "Reference" "C3" (id 0) (at 90.17 52.07 90))
-    (property "Value" "0603" (id 1) (at 93.2561 57.15 90)
-      (effects (font (size 1.27 1.27)) hide)
-    )
-    (property "Footprint" "Capacitor_SMD:C_0603_1608Metric_Pad1.08x0.95mm_HandSolder" (id 2) (at 92.71 53.34 0)
-      (effects (font (size 1.27 1.27)) hide)
-    )
-    (property "Datasheet" "~" (id 3) (at 92.71 53.34 0)
+  (symbol (lib_id "Device:C_Polarized_Small") (at 93.98 53.34 270) (unit 1)
+    (in_bom yes) (on_board yes)
+    (property "Reference" "C3" (id 0) (at 91.44 52.07 90))
+    (property "Value" "10uF" (id 1) (at 97.79 54.61 90))
+    (property "Footprint" "Capacitor_SMD:C_0603_1608Metric_Pad1.08x0.95mm_HandSolder" (id 2) (at 93.98 53.34 0)
+      (effects (font (size 1.27 1.27)) hide)
+    )
+    (property "Datasheet" "~" (id 3) (at 93.98 53.34 0)
       (effects (font (size 1.27 1.27)) hide)
     )
@@
   (symbol (lib_id "Device:C_Small") (at 96.52 49.53 90) (unit 1)
     (in_bom yes) (on_board yes)
-    (property "Reference" "C10" (id 0) (at 93.98 48.26 90))
-    (property "Value" "10pF" (id 1) (at 90.17 48.26 90))
+    (property "Reference" "C10" (id 0) (at 92.71 45.72 90))
+    (property "Value" "10pF" (id 1) (at 92.71 48.26 90))
     (property "Footprint" "Resistor_SMD:R_0402_1005Metric_Pad0.72x0.64mm_HandSolder" (id 2) (at 96.52 49.53 0)
       (effects (font (size 1.27 1.27)) hide)
@@
   )
   (symbol (lib_id "Interface_USB:CH340C") (at 104.14 69.85 0) (unit 1)
-    (in_bom yes) (on_board yes) (fields_autoplaced)
+    (in_bom yes) (on_board yes)
     (property "Reference" "U2" (id 0) (at 106.1594 85.09 0)
       (effects (font (size 1.27 1.27)) (justify left))
@@
   )
   (symbol (lib_id "Regulator_Linear:AMS1117-3.3") (at 72.39 46.99 0) (unit 1)
-    (in_bom yes) (on_board yes) (fields_autoplaced)
+    (in_bom yes) (on_board yes)
     (property "Reference" "U1" (id 0) (at 72.39 39.37 0))
     (property "Value" "AMS1117-3.3" (id 1) (at 72.39 41.91 0))
@@
     (in_bom yes) (on_board yes)
     (property "Reference" "C8" (id 0) (at 80.01 53.34 90))
-    (property "Value" "10pF" (id 1) (at 83.82 57.15 90))
+    (property "Value" "10pF" (id 1) (at 83.82 53.34 90))
     (property "Footprint" "Resistor_SMD:R_0402_1005Metric_Pad0.72x0.64mm_HandSolder" (id 2) (at 77.47 54.61 0)
       (effects (font (size 1.27 1.27)) hide)
@@
     )
     (path "/32201266-c8d7-4d68-abab-ed38d0b5536e"
-      (reference "C3") (unit 1) (value "0603") (footprint "Capacitor_SMD:C_0603_1608Metric_Pad1.08x0.95mm_HandSolder")
+      (reference "C3") (unit 1) (value "10uF") (footprint "Capacitor_SMD:C_0603_1608Metric_Pad1.08x0.95mm_HandSolder")
     )
     (path "/30d3dacd-4777-4fcb-ba43-580b979785c7"
-      (reference "C4") (unit 1) (value "0805") (footprint "Capacitor_SMD:C_0805_2012Metric_Pad1.18x1.45mm_HandSolder")
+      (reference "C4") (unit 1) (value "10uF") (footprint "Capacitor_SMD:C_0805_2012Metric_Pad1.18x1.45mm_HandSolder")
     )
     (path "/c132144a-dea4-4cfc-b78f-82f08cb596a9"
